File: Schematic/Attiny bot.sch (EAGLE design)
At the start: 36 parts, among them IC1 L293D, Q1 SUP65P06-20

Commit message: Schematic of cing
Making it look decent
Parts:
- added R11: 10k, rcl:R-EU_R1206
- added S2: (no value), switch-omron:10-XX
- added SP1: AL11P, buzzer:AL11P
- R1, R3, R4, R5: value (none) -> 10k
Connections:
- removed net N$7: S1.S, S1.S1
- new net BUTTON: R11.2, S2.P, S2.P1, U$1.A6
- new net N$15: SP1.2, U$1.A7
- net +5V: now also S2.S, S2.S1
- net GND: now also R11.1, SP1.1
- net RESET: now also S1.S, S1.S1
Other:
- moved on the sheet: C3, IC1, JP2, JP3, JP4, JP5, JP8, R1, R10, R3, R4, R5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

Commit message: Add files via upload
Parts:
- removed JP2, JP3, JP4, JP5: (no value), pinhead:PINHD-1X3
- removed JP6, JP7: (no value), pinhead:PINHD-1X2
- added JP1-L1, JP2-L2, LIGHTSENSOR1, LIGHTSENSOR2: (no value), pinhead:PINHD-1X3
- added LI-ION-3.7V: 2200MA, diy-modules:BATTERY-LI-MH12210
- added MOT_A, MOT_B: (no value), con-ptr500:AK500/2
- added U$3: USB-SERIAL-FT232R, diy-modules:USB-SERIAL-FT232R
- JP1: value (none) -> indexpin; device pinhead:PINHD-1X2 -> pinhead:PINHD-1X1
- R2: value (none) -> 10k
Connections:
- removed net N$5: C1.2, C2.2, QF1.2
- new net N$16: U$1.D0, U$3.TX
- new net N$7: U$1.D1, U$3.RX
- net +5V: now also LIGHTSENSOR1.2, LIGHTSENSOR2.2; no longer JP2.2, JP3.2
- net A2: now also JP1-L1.2; no longer JP5.2
- net A3: now also JP1.1, JP2-L2.2; no longer JP4.2
- net BAT+: now also LI-ION-3.7V.BAT+; no longer JP1.1
- net BAT-: now also LI-ION-3.7V.BAT-; no longer JP1.2
- net BUTTON: no longer S2.P
- net GND: now also LIGHTSENSOR1.3, LIGHTSENSOR2.3, U$3.GND; no longer JP2.3, JP3.3, S1.P
- net MOT_A+: now also MOT_A-2.KL; no longer JP7.1
- net MOT_A-: now also MOT_A-1.KL; no longer JP7.2
- net MOT_B+: now also MOT_B-2.KL; no longer JP6.1
- net MOT_B-: now also MOT_B-1.KL; no longer JP6.2
- net N$1: now also JP1-L1.1; no longer JP5.1
- net N$12: now also JP2-L2.1; no longer JP4.1
- net N$13: now also JP1-L1.3; no longer JP5.3
- net N$3: now also C2.2
- net N$4: now also C1.2
- net N$6: now also LIGHTSENSOR2.1; no longer JP3.1
- net N$8: now also LIGHTSENSOR1.1; no longer JP2.1
- net N$9: now also JP2-L2.3; no longer JP4.3
- net RESET: no longer S1.S
Other:
- note added: "Connectors"
- note added: "Motor driver"
- note added: "Power managment"
- note added: "Procesor"
- moved on the sheet: C1, C2, C3, C4, C5, C6, C7, C8, D1, D2, IC1, ISP1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
