File: Schematic/procesor-attiny84.brd (EAGLE design)
At the start: 27.9 x 27.9 mm, 5 parts

Commit message: Add files via upload
Parts:
- added E$2: (no value), pinhead:1X01
- moved E$1 0.50 mm to (0.00, 0.77)
Routing:
- net S$7: track 6.13 -> 9.75 mm
- net S$6: track 9.72 -> 12.5 mm
- net S$3: track 15.2 -> 17.5 mm, vias 0 -> 3
- net S$10: track 9.42 -> 8.66 mm
- net S$8: track 13.5 -> 12.8 mm, vias 0 -> 2
- net S$13: track 23.2 -> 22.5 mm, vias 1 -> 0
- net S$14: track 19.9 -> 20.5 mm
- net S$4: track 20.3 -> 19.8 mm
- net S$2: track 12.7 -> 13.2 mm
- net S$15: track 14.3 -> 14.2 mm, vias 1 -> 2
