File: Schematic/esp8266.brd (EAGLE design)
At the start: 35.5 x 37.8 mm, 13 parts, among them IC1 LM1117IMPX-3.3

Commit message: Add files via upload
Routing:
- net +3V3: track 60.9 -> 59.9 mm
Changed lines of the file:
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@@
 <wire x1="46.99" y1="22.09289375" x2="46.99" y2="27.94" width="0.4064" layer="1"/>
 <wire x1="47.7956" y1="21.28729375" x2="46.99" y2="22.09289375" width="0.4064" layer="1"/>
-<wire x1="46.99" y1="27.94" x2="46.355" y2="27.178" width="0.4064" layer="1"/>
-<wire x1="46.355" y1="27.178" x2="45.593" y2="26.797" width="0.4064" layer="1"/>
-<via x="45.593" y="26.797" extent="1-16" drill="0.35"/>
-<wire x1="45.593" y1="26.797" x2="45.009" y2="27.889" width="0.4064" layer="16"/>
+<wire x1="46.99" y1="27.94" x2="46.99" y2="28.067" width="0.4064" layer="1"/>
+<wire x1="46.99" y1="28.067" x2="45.593" y2="28.067" width="0.4064" layer="1"/>
+<via x="45.593" y="28.067" extent="1-16" drill="0.35"/>
+<wire x1="45.593" y1="28.067" x2="45.009" y2="27.889" width="0.4064" layer="16"/>
 <wire x1="45.009" y1="27.889" x2="45.009" y2="27.94" width="0.4064" layer="16"/>
 <wire x1="44.84" y1="36.04" x2="45.8844" y2="34.9956" width="0.4064" layer="1"/>
