File: Hardware/Schematics/Procesors/Procesor-Atmega32u4.brd (EAGLE design)
At the start: 27.5 x 27.5 mm, 5 parts

Commit message: commit
Other:
- board text added: "Sponsored"
- board text added: "by JLCPCB"
Changed lines of the file:
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@@
 <wire x1="-13.5" y1="-14" x2="-13.5" y2="12" width="0" layer="20"/>
 <text x="5.08" y="-5.1" size="1.4" layer="22" rot="MR225" align="center-left">Atmega32u4</text>
+<text x="0" y="7.78" size="1.4" layer="22" rot="MR0" align="bottom-center">Sponsored </text>
+<text x="0" y="5.48" size="1.4" layer="22" rot="MR0" align="bottom-center">by JLCPCB</text>
 </plain>
 <attributes>
