File: Hardware/Schematics/Procesors/Procesor-Attiny85.brd (EAGLE design)
At the start: 27.9 x 27.9 mm, 6 parts

Commit message: commit
Parts:
- added E$2: (no value), atmel:8S1
Connections:
- net S$10: now also E$2.6
- net S$2: now also E$2.1
- net S$3: now also E$2.4
- net S$4: now also E$2.8
- net S$5: now also E$2.7
- net S$6: now also E$2.3
- net S$7: now also E$2.2
- net S$8: now also E$2.5
Routing:
- net S$4: track 26.5 -> 44.3 mm
- net S$3: track 8.67 -> 26.5 mm
- net S$5: track 17.0 -> 23.3 mm
- net S$6: track 24.7 -> 31.0 mm
- net S$10: track 13.8 -> 17.7 mm
- net S$7: track 19.6 -> 23.6 mm
- net S$8: track 8.67 -> 11.1 mm
- net S$2: track 10.2 -> 12.5 mm
Other:
- board size 27.9 x 27.9 mm -> 27.3 x 27.3 mm
- board text added: "Attiny85"
Changed lines of the file:
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@@
 <?xml version="1.0" encoding="utf-8"?>
 <!DOCTYPE eagle SYSTEM "eagle.dtd">
-<eagle version="9.1.0">
+<eagle version="9.2.2">
 <drawing>
 <settings>
-<setting alwaysvectorfont="yes"/>
+<setting alwaysvectorfont="no"/>
 <setting keepoldvectorfont="yes"/>
 <setting verticaltext="up"/>
@@
 <board>
 <plain>
-<wire x1="-13.97" y1="13.97" x2="-13.97" y2="-13.97" width="0.4064" layer="20"/>
-<wire x1="-13.97" y1="-13.97" x2="13.97" y2="-13.97" width="0.4064" layer="20"/>
-<wire x1="13.97" y1="-13.97" x2="13.97" y2="13.97" width="0.4064" layer="20"/>
-<wire x1="13.97" y1="13.97" x2="-13.97" y2="13.97" width="0.4064" layer="20"/>
+<wire x1="-13.67" y1="12.7" x2="-13.67" y2="-13.67" width="0.4064" layer="20"/>
+<wire x1="-13.67" y1="-13.67" x2="13.67" y2="-13.67" width="0.4064" layer="20"/>
+<wire x1="13.67" y1="-13.67" x2="13.67" y2="13.67" width="0.4064" layer="20"/>
+<wire x1="13.67" y1="13.67" x2="-12.7" y2="13.67" width="0.4064" layer="20"/>
+<wire x1="-13.67" y1="12.7" x2="-12.7" y2="13.67" width="0.4064" layer="20"/>
+<text x="0" y="7.62" size="1.778" layer="21" align="center">Attiny85</text>
+<text x="0" y="7.62" size="1.778" layer="22" rot="MR0" align="center">Attiny85</text>
 </plain>
 <attributes>
@@
 </class>
 </classes>
-<designrules name="default">
+<designrules name="default *">
 <description language="de">&lt;b&gt;EAGLE Design Rules&lt;/b&gt;
 &lt;p&gt;
@@
 <param name="mdViaViaSameLayer" value="8mil"/>
 <param name="mnLayersViaInSmd" value="2"/>
-<param name="mdCopperDimension" value="40mil"/>
+<param name="mdCopperDimension" value="10mil"/>
 <param name="mdDrill" value="8mil"/>
 <param name="mdSmdStop" value="0mil"/>
@@
 </autorouter>
 <elements>
-<element name="E$9" library="pinhead" package="1X08" value="" x="-11.43" y="0" rot="R90"/>
-<element name="E$10" library="pinhead" package="1X08" value="" x="0" y="11.43" rot="R180"/>
-<element name="E$11" library="pinhead" package="1X08" value="" x="11.43" y="0" rot="R270"/>
-<element name="E$12" library="pinhead" package="1X08" value="" x="0" y="-11.43"/>
-<element name="ATTINY85" library="atmel" package="DIL08" value="" x="0" y="0" rot="R270"/>
-<element name="E$1" library="pinhead" library_urn="urn:adsk.eagle:library:325" package="1X01" package3d_urn="urn:adsk.eagle:package:22485/2" value="" x="-11.43" y="11.43"/>
+<element name="E$9" library="pinhead" package="1X08" value="" x="-11.43" y="0" smashed="yes" rot="R90">
+<attribute name="VALUE" x="-8.255" y="-10.16" size="1.27" layer="27" rot="R90"/>
+</element>
+<element name="E$10" library="pinhead" package="1X08" value="" x="0" y="11.43" smashed="yes" rot="R180">
+<attribute name="VALUE" x="10.16" y="14.605" size="1.27" layer="27" rot="R180"/>
+</element>
+<element name="E$11" library="pinhead" package="1X08" value="" x="11.43" y="0" smashed="yes" rot="R270">
+<attribute name="VALUE" x="8.255" y="10.16" size="1.27" layer="27" rot="R270"/>
+</element>
+<element name="E$12" library="pinhead" package="1X08" value="" x="0" y="-11.43" smashed="yes">
+<attribute name="VALUE" x="-10.16" y="-14.605" size="1.27" layer="27"/>
+</element>
+<element name="ATTINY85" library="atmel" package="DIL08" value="" x="0" y="0" smashed="yes" rot="R270">
+<attribute name="VALUE" x="-0.9906" y="3.81" size="1.27" layer="27" ratio="10" rot="R270"/>
+</element>
+<element name="E$1" library="pinhead" library_urn="urn:adsk.eagle:library:325" package="1X01" package3d_urn="urn:adsk.eagle:package:22485/2" value="" x="-11.43" y="11.43" smashed="yes">
+<attribute name="VALUE" x="-12.7" y="8.255" size="1.27" layer="27"/>
+</element>
+<element name="E$2" library="atmel" library_urn="urn:adsk.eagle:library:105" package="8S1" package3d_urn="urn:adsk.eagle:package:4358/1" value="" x="0" y="0" smashed="yes" rot="MR180">
+<attribute name="VALUE" x="4.064" y="2.159" size="1.27" layer="28" ratio="10" rot="MR270"/>
+</element>
 </elements>
 <signals>
@@
 <wire x1="-3.81" y1="8.89" x2="-1.27" y2="8.89" width="0.8128" layer="1"/>
 <wire x1="-1.27" y1="8.89" x2="-1.27" y2="11.43" width="0.8128" layer="1"/>
+<contactref element="E$2" pad="1"/>
+<wire x1="-1.905" y1="2.654" x2="-2.654" y2="2.654" width="0.4064" layer="16"/>
+<wire x1="-2.654" y1="2.654" x2="-3.81" y2="3.81" width="0.4064" layer="16"/>
 </signal>
 <signal name="S$3">
@@
 <wire x1="-6.35" y1="-3.81" x2="-8.89" y2="-1.27" width="0.8128" layer="1"/>
 <wire x1="-8.89" y1="-1.27" x2="-11.43" y2="-1.27" width="0.8128" layer="1"/>
+<contactref element="E$2" pad="4"/>
+<wire x1="-3.81" y1="-3.051" x2="-3.81" y2="-3.81" width="0.4064" layer="16"/>
+<wire x1="-4.9122875" y1="4.8768" x2="-5.5372" y2="4.2518875" width="0.4064" layer="16"/>
+<wire x1="-5.5372" y1="-1.7118875" x2="-4.9122875" y2="-2.3368" width="0.4064" layer="16"/>
+<wire x1="1.895" y1="2.654" x2="1.3314" y2="3.2176" width="0.4064" layer="16"/>
+<wire x1="1.3314" y1="3.2176" x2="1.3314" y2="3.6223375" width="0.4064" layer="16"/>
+<wire x1="-4.9122875" y1="-2.3368" x2="-4.5242" y2="-2.3368" width="0.4064" layer="16"/>
+<wire x1="-4.5242" y1="-2.3368" x2="-3.81" y2="-3.051" width="0.4064" layer="16"/>
+<wire x1="1.3314" y1="3.6223375" x2="0.0769375" y2="4.8768" width="0.4064" layer="16"/>
+<wire x1="0.0769375" y1="4.8768" x2="-4.9122875" y2="4.8768" width="0.4064" layer="16"/>
+<wire x1="-5.5372" y1="4.2518875" x2="-5.5372" y2="-1.7118875" width="0.4064" layer="16"/>
 </signal>
 <signal name="S$4">
@@
 <wire x1="1.27" y1="-6.35" x2="1.27" y2="3.81" width="0.8128" layer="1"/>
 <wire x1="1.27" y1="3.81" x2="3.81" y2="3.81" width="0.8128" layer="1"/>
+<contactref element="E$2" pad="8"/>
+<wire x1="3.81" y1="3.061" x2="3.81" y2="3.81" width="0.4064" layer="16"/>
+<wire x1="4.9122875" y1="-4.8768" x2="5.5372" y2="-4.2518875" width="0.4064" layer="16"/>
+<wire x1="5.5372" y1="1.7118875" x2="4.9122875" y2="2.3368" width="0.4064" layer="16"/>
+<wire x1="-1.905" y1="-2.654" x2="-1.3414" y2="-3.2176" width="0.4064" layer="16"/>
+<wire x1="-1.3414" y1="-3.2176" x2="-1.3414" y2="-3.6223375" width="0.4064" layer="16"/>
+<wire x1="4.9122875" y1="2.3368" x2="4.5342" y2="2.3368" width="0.4064" layer="16"/>
+<wire x1="4.5342" y1="2.3368" x2="3.81" y2="3.061" width="0.4064" layer="16"/>
+<wire x1="-1.3414" y1="-3.6223375" x2="-0.0869375" y2="-4.8768" width="0.4064" layer="16"/>
+<wire x1="-0.0869375" y1="-4.8768" x2="4.9122875" y2="-4.8768" width="0.4064" layer="16"/>
+<wire x1="5.5372" y1="-4.2518875" x2="5.5372" y2="1.7118875" width="0.4064" layer="16"/>
 </signal>
 <signal name="S$6">
@@
 <wire x1="7.62" y1="8.89" x2="8.89" y2="10.16" width="0.8128" layer="1"/>
 <wire x1="8.89" y1="10.16" x2="8.89" y2="11.43" width="0.8128" layer="1"/>
+<contactref element="E$2" pad="3"/>
+<wire x1="0.625" y1="2.654" x2="0.0614" y2="2.0904" width="0.4064" layer="16"/>
+<wire x1="0.0614" y1="2.0904" x2="0.0614" y2="1.6856625" width="0.4064" layer="16"/>
+<wire x1="0.0614" y1="1.6856625" x2="-2.8942625" y2="-1.27" width="0.4064" layer="16"/>
+<wire x1="-2.8942625" y1="-1.27" x2="-3.81" y2="-1.27" width="0.4064" layer="16"/>
 </signal>
 <signal name="S$7">
@@
 <wire x1="-1.27" y1="7.62" x2="6.35" y2="7.62" width="0.8128" layer="1"/>
 <wire x1="6.35" y1="7.62" x2="6.35" y2="11.43" width="0.8128" layer="1"/>
+<contactref element="E$2" pad="2"/>
+<wire x1="-0.645" y1="2.654" x2="-1.1986" y2="2.1004" width="0.4064" layer="16"/>
+<wire x1="-1.1986" y1="2.1004" x2="-1.1986" y2="1.6856625" width="0.4064" layer="16"/>
+<wire x1="-1.1986" y1="1.6856625" x2="-1.6142625" y2="1.27" width="0.4064" layer="16"/>
+<wire x1="-1.6142625" y1="1.27" x2="-3.81" y2="1.27" width="0.4064" layer="16"/>
 </signal>
 <signal name="S$5">
@@
 <wire x1="8.89" y1="-7.62" x2="10.16" y2="-8.89" width="0.8128" layer="1"/>
 <wire x1="10.16" y1="-8.89" x2="11.43" y2="-8.89" width="0.8128" layer="1"/>
+<contactref element="E$2" pad="7"/>
+<wire x1="-0.635" y1="-2.654" x2="-0.0714" y2="-2.0904" width="0.4064" layer="16"/>
+<wire x1="-0.0714" y1="-2.0904" x2="-0.0714" y2="-1.6856625" width="0.4064" layer="16"/>
+<wire x1="-0.0714" y1="-1.6856625" x2="2.8842625" y2="1.27" width="0.4064" layer="16"/>
+<wire x1="2.8842625" y1="1.27" x2="3.81" y2="1.27" width="0.4064" layer="16"/>
 </signal>
 <signal name="S$8">
@@
 <wire x1="3.81" y1="-7.62" x2="6.35" y2="-10.16" width="0.8128" layer="1"/>
 <wire x1="6.35" y1="-10.16" x2="6.35" y2="-11.43" width="0.8128" layer="1"/>
+<contactref element="E$2" pad="5"/>
+<wire x1="1.905" y1="-2.654" x2="3.061" y2="-3.81" width="0.4064" layer="16"/>
+<wire x1="3.061" y1="-3.81" x2="3.81" y2="-3.81" width="0.4064" layer="16"/>
 </signal>
 <signal name="S$10">
@@
 <wire x1="6.35" y1="-7.62" x2="6.35" y2="-1.27" width="0.8128" layer="1"/>
 <wire x1="6.35" y1="-1.27" x2="3.81" y2="-1.27" width="0.8128" layer="1"/>
+<contactref element="E$2" pad="6"/>
+<wire x1="0.635" y1="-2.654" x2="1.1986" y2="-2.0904" width="0.4064" layer="16"/>
+<wire x1="1.1986" y1="-2.0904" x2="1.1986" y2="-1.6856625" width="0.4064" layer="16"/>
+<wire x1="1.1986" y1="-1.6856625" x2="1.6142625" y2="-1.27" width="0.4064" layer="16"/>
+<wire x1="1.6142625" y1="-1.27" x2="3.81" y2="-1.27" width="0.4064" layer="16"/>
 </signal>
 </signals>

Commit message: commit
Other:
- board text added: "Sponsored by JLCPCB"
Changed lines of the file:
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@@
 <text x="0" y="7.62" size="1.778" layer="21" align="center">Attiny85</text>
 <text x="0" y="7.62" size="1.778" layer="22" rot="MR0" align="center">Attiny85</text>
+<text x="0" y="-7.62" size="1.016" layer="21" align="center">Sponsored by JLCPCB</text>
 </plain>
 <attributes>

Commit message: gerber update
Other:
- board text removed: "Sponsored by JLCPCB"
Changed lines of the file:
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@@
 <?xml version="1.0" encoding="utf-8"?>
 <!DOCTYPE eagle SYSTEM "eagle.dtd">
-<eagle version="9.2.2">
+<eagle version="9.4.0">
 <drawing>
 <settings>
@@
 <text x="0" y="7.62" size="1.778" layer="21" align="center">Attiny85</text>
 <text x="0" y="7.62" size="1.778" layer="22" rot="MR0" align="center">Attiny85</text>
-<text x="0" y="-7.62" size="1.016" layer="21" align="center">Sponsored by JLCPCB</text>
 </plain>
 <attributes>

Commit message: 3D package upgrade
Parts:
- flipped E$1 to the bottom
- flipped E$10 to the bottom, turned to 0 degrees
- flipped E$11 to the bottom
- flipped E$12 to the bottom, turned to 180 degrees
- flipped E$9 to the bottom
