File: Hardware/Schematics/Procesors/Procesor-ESP8266.brd (EAGLE design)
At the start: 35.5 x 37.8 mm, 7 parts

Commit message: commit
Parts:
- moved J3 49.3 mm to (-6.35, -11.4)
- moved J4 49.3 mm to (14.0, -8.89)
- moved U1 49.3 mm to (0.00, 0.00)
- moved J1 49.3 mm to (11.4, 11.4)
- moved J2 49.3 mm to (-8.89, 8.89)
- moved JP5 49.3 mm to (-8.89, 11.4)
- moved TP1 49.3 mm to (2.54, 11.4)
Routing:
- net GND: track 28.0 -> 48.2 mm, vias 1 -> 2
- net A2: track 15.3 -> 12.2 mm
- net A5: track 27.6 -> 26.9 mm
- net A6: track 27.1 -> 27.8 mm
- net +5V: track 52.4 -> 51.8 mm
- net A4: track 15.7 -> 15.2 mm
Other:
- board size 35.5 x 37.8 mm -> 34 x 34 mm
- board text added: "ESP 8266"
- board text removed: "Cing"
- board text removed: "ESP 8266 OTA"

Commit message: 3D package upgrade
Parts:
- flipped JP5 to the top
Changed lines of the file:
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@@
 <?xml version="1.0" encoding="utf-8"?>
 <!DOCTYPE eagle SYSTEM "eagle.dtd">
-<eagle version="9.2.2">
+<eagle version="9.4.0">
 <drawing>
 <settings>
-<setting alwaysvectorfont="no"/>
+<setting alwaysvectorfont="yes"/>
 <setting verticaltext="up"/>
 </settings>
@@
 </layers>
 <board>
+<fusionsync huburn="a.cGVyc29uYWw6dWUyOTc5YzVj" projecturn="a.cGVyc29uYWw6dWUyOTc5YzVjIzIwMTkwNjI1MjAwNjYyNTAx" f3durn="urn:adsk.wipprod:dm.lineage:gThltiGNS-Os0w2pd-l9LA" pcbguid="ef190aa2-9681-48f3-8ae9-ed52396e28e6" lastpulledtime="" lastsyncedchangeguid="f7c9b0ec-481d-b649-d203-f000a8791a48"/>
 <plain>
 <wire x1="-16" y1="-17" x2="18" y2="-17" width="0" layer="20"/>
@@
 </autorouter>
 <elements>
-<element name="JP5" library="pinhead" library_urn="urn:adsk.eagle:library:325" package="1X01" package3d_urn="urn:adsk.eagle:package:22485/2" value="" x="-8.89" y="11.43" smashed="yes" rot="MR0">
-<attribute name="VALUE" x="-7.62" y="8.255" size="1.27" layer="28" rot="MR0"/>
+<element name="JP5" library="pinhead" library_urn="urn:adsk.eagle:library:325" package="1X01" package3d_urn="urn:adsk.eagle:package:22485/2" value="" x="-8.89" y="11.43" smashed="yes">
+<attribute name="VALUE" x="-10.16" y="8.255" size="1.27" layer="27"/>
 </element>
 <element name="TP1" library="testpad" library_urn="urn:adsk.eagle:library:385" package="B1,27" package3d_urn="urn:adsk.eagle:package:27944/1" value="PTR1B1,27" x="2.54" y="11.43" smashed="yes">
@@
 <attribute name="VALUE" x="1.905" y="10.668" size="0.0254" layer="27"/>
 </element>
-<element name="U1" library="esp12e" package="ESP12E-SMD" value="" x="0" y="0" smashed="yes" rot="R90">
+<element name="U1" library="esp12e" package="ESP12E-SMD" override_package3d_urn="urn:adsk.eagle:package:11842534/2" override_package_urn="urn:adsk.eagle:footprint:11842537/1" value="" x="0" y="0" smashed="yes" rot="R90">
 <attribute name="VALUE" x="11.9" y="-7.7" size="1.4224" layer="27" rot="R90"/>
 </element>
@@
 <polygon width="2.54" layer="1">
 <vertex x="-13.97" y="48.26"/>
-<vertex x="-13.97" y="48.26"/>
 <vertex x="24.13" y="48.26"/>
 <vertex x="24.13" y="-17.30375"/>
@@
 </note>
 <note version="8.3" severity="warning">
+Since Version 8.3, EAGLE supports Fusion synchronisation.
+This feature will not be available in this version and saving
+the document will break the link to the Fusion PCB feature.
+</note>
+<note version="8.3" severity="warning">
 Since Version 8.3, EAGLE supports URNs for individual library
 assets (packages, symbols, and devices). The URNs of those assets
@@
 packages will not be understood (or retained) with this version.
 </note>
+<note version="9.4" severity="warning">
+Since Version 9.4, EAGLE supports the overriding of 3D packages
+in schematics and board files. Those overridden 3d packages
+will not be understood (or retained) with this version.
+</note>
 </compatibility>
