File: Hardware/Schematics/Procesors/Procesor-Attiny84.brd (EAGLE design)
At the start: 27.9 x 27.9 mm, 6 parts

Commit message: commit
Parts:
- added E$3: (no value), SparkFun-IC-Microcontroller:SO14
- moved E$1 3.54 mm to (3.50, 0.27)
Connections:
- net S$10: now also E$3.8
- net S$11: now also E$3.10
- net S$12: now also E$3.11
- net S$13: now also E$3.2
- net S$14: now also E$3.3
- net S$15: now also E$3.5
- net S$18: now also E$3.6
- net S$2: now also E$3.4
- net S$3: now also E$3.14
- net S$4: now also E$3.1
- net S$5: now also E$3.9
- net S$6: now also E$3.12
- net S$7: now also E$3.13
- net S$8: now also E$3.7
Routing:
- net S$3: track 10.6 -> 37.1 mm
- net S$7: track 9.75 -> 29.9 mm
- net S$5: track 9.39 -> 24.6 mm
- net S$6: track 12.5 -> 27.6 mm
- net S$10: track 8.66 -> 23.1 mm
- net S$12: track 8.75 -> 22.5 mm
- net S$8: track 13.7 -> 27.1 mm
- net S$11: track 8.34 -> 21.6 mm
- net S$4: track 19.8 -> 25.9 mm
- net S$13: track 22.5 -> 27.4 mm
- net S$15: track 14.0 -> 18.7 mm
- net S$2: track 13.2 -> 15.4 mm
- net S$14: track 20.5 -> 22.4 mm
- net S$18: track 10.9 -> 12.7 mm
Other:
- board size 27.9 x 27.9 mm -> 27.3 x 27.3 mm
- board text added: "Attiny84"

Commit message: commit
Other:
- board text added: "Sponsored"
- board text added: "by JLCPCB"
Changed lines of the file:
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@@
 <text x="3.5" y="0.5" size="1.778" layer="21" rot="R90" align="center">Attiny84</text>
 <text x="3.5" y="0.5" size="1.778" layer="22" rot="MR90" align="center">Attiny84</text>
+<text x="-7" y="0" size="1.778" layer="21" rot="R270" align="bottom-center">Sponsored</text>
+<text x="-4.5" y="0.5" size="1.778" layer="21" rot="R270" align="bottom-center">by JLCPCB</text>
 </plain>
 <attributes>

Commit message: gerber update
Other:
- outline, holes or cut-outs redrawn
- board text removed: "Sponsored"
- board text removed: "by JLCPCB"
Changed lines of the file:
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@@
 <?xml version="1.0" encoding="utf-8"?>
 <!DOCTYPE eagle SYSTEM "eagle.dtd">
-<eagle version="9.2.2">
+<eagle version="9.4.0">
 <drawing>
 <settings>
@@
 <board>
 <plain>
-<wire x1="-13.67" y1="12.7" x2="-12.7" y2="13.67" width="0.4064" layer="20"/>
-<wire x1="-12.7" y1="13.67" x2="13.67" y2="13.67" width="0.4064" layer="20"/>
+<wire x1="-13.67" y1="12.2" x2="-12.2" y2="13.67" width="0.4064" layer="20"/>
+<wire x1="-12.2" y1="13.67" x2="13.67" y2="13.67" width="0.4064" layer="20"/>
 <wire x1="13.67" y1="13.67" x2="13.67" y2="-13.67" width="0.4064" layer="20"/>
 <wire x1="13.67" y1="-13.67" x2="-13.67" y2="-13.67" width="0.4064" layer="20"/>
-<wire x1="-13.67" y1="-13.67" x2="-13.67" y2="12.7" width="0.4064" layer="20"/>
+<wire x1="-13.67" y1="-13.67" x2="-13.67" y2="12.2" width="0.4064" layer="20"/>
 <text x="3.5" y="0.5" size="1.778" layer="21" rot="R90" align="center">Attiny84</text>
 <text x="3.5" y="0.5" size="1.778" layer="22" rot="MR90" align="center">Attiny84</text>
-<text x="-7" y="0" size="1.778" layer="21" rot="R270" align="bottom-center">Sponsored</text>
-<text x="-4.5" y="0.5" size="1.778" layer="21" rot="R270" align="bottom-center">by JLCPCB</text>
 </plain>
 <attributes>

Commit message: 3D package upgrade
Parts:
- moved E$10 0.14 mm to (0.00, 11.6), flipped to the bottom, turned to 0 degrees
- flipped E$11 to the bottom
- flipped E$12 to the bottom, turned to 180 degrees
- flipped E$2 to the bottom
- flipped E$9 to the bottom
Routing:
- net S$8: track 27.1 -> 26.4 mm

Commit message: gerber update
Routing:
- net S$3: track 37.1 -> 35.2 mm
- net S$8: track 26.4 -> 24.9 mm
- net S$4: track 25.9 -> 24.8 mm
- net S$7: track 30.0 -> 29.1 mm
Changed lines of the file:
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@@
 <text x="3.5" y="0.5" size="1.778" layer="21" rot="R90" align="center">Attiny84</text>
 <text x="3.5" y="0.5" size="1.778" layer="22" rot="MR90" align="center">Attiny84</text>
+<text x="-6" y="0" size="1.778" layer="21" rot="R90" align="center">Attiny84</text>
 </plain>
 <attributes>
@@
 <contactref element="E$3" pad="4"/>
 <wire x1="1" y1="1.58" x2="-0.31" y2="0.27" width="0.254" layer="1"/>
-<wire x1="1" y1="9.16" x2="1" y2="9" width="0.254" layer="1"/>
 <wire x1="1" y1="9" x2="1" y2="1.58" width="0.254" layer="1"/>
 <wire x1="-3.015" y1="0.055" x2="-0.525" y2="0.055" width="0.254" layer="16"/>
 <wire x1="-0.525" y1="0.055" x2="-0.31" y2="0.27" width="0.254" layer="16"/>
-<wire x1="1" y1="9" x2="-1.27" y2="11.27" width="0.254" layer="1"/>
+<wire x1="-1.27" y1="11.27" x2="1" y2="9" width="0.254" layer="1"/>
 <wire x1="-1.27" y1="11.27" x2="-1.27" y2="11.57" width="0.254" layer="1"/>
 </signal>
@@
 <wire x1="-0.31" y1="7.89" x2="-2.215" y2="5.985" width="0.254" layer="1"/>
 <wire x1="-2.215" y1="5.985" x2="-7.88303125" y2="5.985" width="0.254" layer="1"/>
-<wire x1="-7.88303125" y1="5.985" x2="-9.5" y2="4.36803125" width="0.254" layer="1"/>
-<wire x1="-9.5" y1="4.36803125" x2="-9.5" y2="-3.81" width="0.254" layer="1"/>
+<wire x1="-9.5" y1="4.36803125" x2="-7.88303125" y2="5.985" width="0.254" layer="1"/>
 <contactref element="E$3" pad="1"/>
 <wire x1="-3.015" y1="3.865" x2="-3.015" y2="5.185" width="0.254" layer="16"/>
 <wire x1="-3.015" y1="5.185" x2="-0.31" y2="7.89" width="0.254" layer="16"/>
-<wire x1="-9.5" y1="-3.81" x2="-11.43" y2="-3.81" width="0.254" layer="1"/>
+<wire x1="-11.43" y1="-3.81" x2="-9.5" y2="-1.88" width="0.254" layer="1"/>
+<wire x1="-9.5" y1="-1.88" x2="-9.5" y2="4.36803125" width="0.254" layer="1"/>
 </signal>
 <signal name="S$6">
@@
 <wire x1="7.31" y1="6.27355" x2="8.453" y2="7.41655" width="0.254" layer="1"/>
 <wire x1="7.31" y1="5.35" x2="7.31" y2="6.19" width="0.254" layer="16"/>
-<wire x1="7.31" y1="6.19" x2="6" y2="7.5" width="0.254" layer="16"/>
-<wire x1="6" y1="7.5" x2="6" y2="9" width="0.254" layer="16"/>
-<wire x1="6" y1="9" x2="0.19645" y2="9" width="0.254" layer="16"/>
-<wire x1="0.19645" y1="9" x2="0.16345" y2="9.033" width="0.254" layer="16"/>
 <wire x1="-7.22145" y1="4.61196875" x2="-7.22145" y2="3" width="0.254" layer="16"/>
-<wire x1="0.16345" y1="9.033" x2="-2.80041875" y2="9.033" width="0.254" layer="16"/>
 <wire x1="-2.80041875" y1="9.033" x2="-7.22145" y2="4.61196875" width="0.254" layer="16"/>
 <wire x1="-7.22145" y1="3" x2="-7.62645" y2="2.595" width="0.254" layer="16"/>
@@
 <wire x1="8.453" y1="7.41655" x2="8.453" y2="9.467" width="0.254" layer="1"/>
 <wire x1="8.453" y1="9.467" x2="6.35" y2="11.57" width="0.254" layer="1"/>
+<wire x1="7.31" y1="6.19" x2="4.467" y2="9.033" width="0.254" layer="16"/>
+<wire x1="4.467" y1="9.033" x2="-2.80041875" y2="9.033" width="0.254" layer="16"/>
 </signal>
 <signal name="S$5">
@@
 <contactref element="E$12" pad="7"/>
 <contactref element="E$1" pad="7"/>
-<wire x1="0" y1="-3.5" x2="-3" y2="-3.5" width="0.254" layer="1"/>
-<wire x1="-3" y1="-3.5" x2="-3" y2="-7.5" width="0.254" layer="1"/>
-<wire x1="-3" y1="-7.5" x2="-0.46" y2="-7.5" width="0.254" layer="1"/>
+<wire x1="0" y1="-3.5" x2="-1.5" y2="-3.5" width="0.254" layer="1"/>
+<wire x1="-0.46" y1="-7.5" x2="-2" y2="-7.5" width="0.254" layer="1"/>
 <wire x1="-0.46" y1="-7.5" x2="-0.31" y2="-7.35" width="0.254" layer="1"/>
 <contactref element="E$3" pad="7"/>
@@
 <wire x1="6.35" y1="-11.43" x2="6.35" y2="-9.85" width="0.254" layer="1"/>
 <wire x1="6.35" y1="-9.85" x2="0" y2="-3.5" width="0.254" layer="1"/>
+<wire x1="-3" y1="-5" x2="-1.5" y2="-3.5" width="0.254" layer="1"/>
+<wire x1="-2" y1="-7.5" x2="-3" y2="-6.5" width="0.254" layer="1"/>
+<wire x1="-3" y1="-6.5" x2="-3" y2="-5" width="0.254" layer="1"/>
 </signal>
 <signal name="S$10">
@@
 <contactref element="E$11" pad="4"/>
 <contactref element="E$1" pad="14"/>
-<wire x1="6.81" y1="7.89" x2="7.31" y2="7.89" width="0.254" layer="1"/>
-<wire x1="4.667" y1="-0.20345" x2="5.33655" y2="-0.873" width="0.254" layer="1"/>
-<wire x1="4.667" y1="5.82345" x2="5.33655" y2="6.493" width="0.254" layer="1"/>
-<wire x1="5.33655" y1="6.493" x2="5.413" y2="6.493" width="0.254" layer="1"/>
-<wire x1="5.413" y1="6.493" x2="6.81" y2="7.89" width="0.254" layer="1"/>
-<wire x1="4.667" y1="-0.20345" x2="4.667" y2="5.82345" width="0.254" layer="1"/>
 <contactref element="E$3" pad="14"/>
 <wire x1="-8.615" y1="3.865" x2="-2.98" y2="9.5" width="0.254" layer="16"/>
@@
 <wire x1="7" y1="8.2" x2="7.31" y2="7.89" width="0.254" layer="16"/>
 <wire x1="9.287" y1="-0.873" x2="11.43" y2="1.27" width="0.254" layer="1"/>
-<wire x1="5.33655" y1="-0.873" x2="9.287" y2="-0.873" width="0.254" layer="1"/>
+<wire x1="9.287" y1="-0.873" x2="6.5" y2="-0.873" width="0.254" layer="1"/>
+<wire x1="5.8135" y1="-0.1865" x2="6.5" y2="-0.873" width="0.254" layer="1"/>
+<wire x1="5.8135" y1="6.3935" x2="5.8135" y2="-0.1865" width="0.254" layer="1"/>
+<wire x1="5.8135" y1="6.3935" x2="7.31" y2="7.89" width="0.254" layer="1"/>
 </signal>
 </signals>
