File: Hardware/Schematics/Sensors/UltrasonicSensor/UltrasonicSensor.brd (EAGLE design)
At the start: 69.5 x 20.4 mm, 19 parts

Commit message: commit
Other:
- board text added: "Sponsored by JLCPCB"
- board text removed: "Ultrasonic Sensor"
- board text removed: "for Robot Cing"
Changed lines of the file:
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@@
 <wire x1="-24.47" y1="-10.6" x2="24.47" y2="-10.6" width="0.0762" layer="20"/>
 <wire x1="24.47" y1="9.83" x2="-24.47" y2="9.83" width="0.0762" layer="20"/>
-<text x="0" y="-4" size="1.27" layer="21" rot="R180" align="bottom-center">Ultrasonic Sensor
+<text x="0" y="-4.4" size="1.27" layer="21" rot="R180" align="bottom-center">Sponsored by JLCPCB
 </text>
-<text x="0" y="-5.5" size="1.27" layer="21" rot="R180" align="bottom-center">for Robot Cing</text>
 <circle x="-4.1" y="-3" radius="0.360553125" width="0.1524" layer="26"/>
 <wire x1="-24.47" y1="-10.6" x2="-24.47" y2="9.83" width="0.0762" layer="20" curve="-180.561665"/>
