File: Hardware/Schematics/Sensors/UltrasonicSensor/UltrasonicSensor.brd (EAGLE design)
At the start: 69.5 x 20.4 mm, 19 parts

Commit message: Patches
Parts:
- removed SJ4: (no value), jumper:SJ
- added R4: 1k, rcl:M1206
- R1, R3: value (none) -> 100R
- R2: value (none) -> 100k
- moved R2 5.00 mm to (10.0, 2.62), flipped to the bottom, turned to 0 degrees
- moved SJ1 4.00 mm to (13.0, 7.20)
- moved SJ3 4.00 mm to (10.8, 7.20)
- moved SJ5 4.00 mm to (8.60, 7.20)
- moved U$8 1.02 mm to (-28.2, 0.00)
- moved U$9 1.02 mm to (28.2, 0.00)
Connections:
- net N$1 renamed 9
- net N$3 renamed 8
- net N$5 renamed 0
- removed net N$4: SJ4.1, U$2.6
- new net N$1: R4.2, U$6.A1
- net GND: no longer SJ4.2
- net OUTPUT: now also R4.1, U$2.6; no longer U$6.A1
Routing:
- net OUTPUT: track 19.5 -> 36.1 mm, vias 0 -> 1
- net N$4: track 6.03 -> 0.00 mm, vias 1 -> 0
- net POT: track 19.4 -> 15.2 mm, vias 2 -> 1
- net N$1: track 0.00 -> 4.02 mm
- net SCL: track 59.6 -> 63.1 mm
- net GND: track 15.9 -> 13.1 mm
- net 0: track 30.9 -> 28.0 mm
- net 8: track 35.3 -> 32.8 mm
- net 9: track 31.8 -> 29.4 mm
Other:
- board text added: "1"
- board text added: "2"
- board text added: "3"

Commit message: commit
Parts:
- flipped U$6 to the bottom
Routing:
- net N$1: track 4.02 -> 13.8 mm
Changed lines of the file:
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@@
 </element>
 <element name="U$5" library="Cing Library" package="OSHW_5MM" value="OPENSOURCE" x="0" y="-2" smashed="yes"/>
-<element name="U$6" library="Cing Library" package="CONNECTOR_1X5" value="CONNECTOR_1X5" x="-13.462" y="-8.63" smashed="yes" rot="R270"/>
+<element name="U$6" library="Cing Library" package="CONNECTOR_1X5" value="CONNECTOR_1X5" x="-13.462" y="-8.63" smashed="yes" rot="MR270"/>
 <element name="SJ1" library="jumper" library_urn="urn:adsk.eagle:library:252" package="SJ" package3d_urn="urn:adsk.eagle:package:15471/1" value="" x="13" y="7.2" smashed="yes" rot="R270">
 <attribute name="VALUE" x="13" y="6.7999" size="0.02" layer="27" rot="R270"/>
@@
 <contactref element="U$6" pad="A1"/>
 <contactref element="R4" pad="2"/>
-<wire x1="-6" y1="-5.6" x2="-8.382" y2="-7.982" width="0.1524" layer="16"/>
-<wire x1="-8.382" y1="-7.982" x2="-8.382" y2="-8.63" width="0.1524" layer="16"/>
+<wire x1="-6" y1="-5.6" x2="-15.512" y2="-5.6" width="0.1524" layer="16"/>
+<wire x1="-15.512" y1="-5.6" x2="-18.542" y2="-8.63" width="0.1524" layer="16"/>
 </signal>
 </signals>

Commit message: gerber update
Other:
- board text added: "I2c"
- board text added: "Trig"
Changed lines of the file:
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@@
 <?xml version="1.0" encoding="utf-8"?>
 <!DOCTYPE eagle SYSTEM "eagle.dtd">
-<eagle version="9.2.2">
+<eagle version="9.4.0">
 <drawing>
 <settings>
-<setting alwaysvectorfont="no"/>
+<setting alwaysvectorfont="yes"/>
 <setting verticaltext="up"/>
 </settings>
@@
 <text x="10.8" y="5.306" size="1.27" layer="21" rot="R180" align="bottom-center">2</text>
 <text x="13" y="5.306" size="1.27" layer="21" rot="R180" align="bottom-center">3</text>
+<text x="7.619" y="-8.9" size="1.27" layer="21" rot="R180" align="bottom-center">Trig</text>
+<text x="25.619" y="-5.9" size="1.27" layer="21" rot="R180" align="bottom-center">I2c</text>
+<text x="-25.619" y="-5.9" size="1.27" layer="21" rot="R180" align="bottom-center">I2c</text>
 </plain>
 <attributes>
@@
 <element name="U$2" library="SparkFun-IC-Microcontroller" library_urn="urn:adsk.eagle:library:525" package="SO14" package3d_urn="urn:adsk.eagle:package:38947/1" value="ATTINY84" x="-0.762" y="-1.905" smashed="yes" rot="MR180">
 <attribute name="PROD_ID" value="IC-11285" x="46.228" y="28.575" size="1.778" layer="28" rot="MR180" display="off"/>
-<attribute name="VALUE" x="5.588" y="-1.905" size="0.8128" layer="28" font="vector" ratio="12" rot="MR270" align="bottom-center"/>
 </element>
 <element name="U$3" library="Cing Library" package="I2_HEADER" value="I2C_HEADER" x="-18.669" y="0" smashed="yes"/>
@@
 <element name="R1" library="rcl" library_urn="urn:adsk.eagle:library:334" package="M1206" package3d_urn="urn:adsk.eagle:package:23566/1" value="100R" x="12.827" y="-1.27" smashed="yes" rot="R90">
 <attribute name="SPICEPREFIX" value="R" x="12.827" y="-1.27" size="1.778" layer="27" rot="R90" display="off"/>
-<attribute name="VALUE" x="15.367" y="-4.54" size="1.27" layer="27" rot="R90"/>
 </element>
 <element name="R3" library="rcl" library_urn="urn:adsk.eagle:library:334" package="M1206" package3d_urn="urn:adsk.eagle:package:23566/1" value="100R" x="10.033" y="-1.27" smashed="yes" rot="R270">
 <attribute name="SPICEPREFIX" value="R" x="10.033" y="-1.27" size="1.778" layer="27" rot="R270" display="off"/>
-<attribute name="VALUE" x="7.62" y="-0.254" size="1.27" layer="27" rot="R270"/>
 </element>
 <element name="LED1" library="led" library_urn="urn:adsk.eagle:library:259" package="CHIPLED_1206" package3d_urn="urn:adsk.eagle:package:15823/2" value="" x="12.7" y="-7.62" smashed="yes">
@@
 <element name="R4" library="rcl" library_urn="urn:adsk.eagle:library:334" package="M1206" package3d_urn="urn:adsk.eagle:package:23566/1" value="1k" x="-6" y="-7" smashed="yes" rot="MR90">
 <attribute name="SPICEPREFIX" value="R" x="-6" y="-7" size="1.778" layer="28" rot="MR90" display="off"/>
-<attribute name="VALUE" x="-6.54" y="-4.27" size="1.27" layer="28" rot="MR90"/>
 </element>
 </elements>
