File: Hardware/Schematics/Sensors/UltrasonicSensor/UltrasonicSensor.sch (EAGLE design)
At the start: 19 parts

Commit message: Patches
Parts:
- removed SJ4: (no value), jumper:SJ
- added R4: 1k, rcl:R-EU_M1206
- R1, R3: value (none) -> 100R
- R2: value (none) -> 100k
Connections:
- net N$1 renamed 9
- net N$3 renamed 8
- net N$5 renamed 0
- removed net N$4: SJ4.1, U$2.(PCINT7/ICP/OC0B/ADC7)PA7
- new net N$1: R4.2, U$6.A1
- net GND: no longer SJ4.2
- net OUTPUT: now also R4.1, U$2.(PCINT7/ICP/OC0B/ADC7)PA7; no longer U$6.A1
Other:
- moved on the sheet: SJ1, SJ3, SJ5
Changed lines of the file:
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@@
 <part name="+3V7" library="supply1" library_urn="urn:adsk.eagle:library:371" deviceset="+3V3" device=""/>
 <part name="GND7" library="supply1" library_urn="urn:adsk.eagle:library:371" deviceset="GND" device=""/>
-<part name="R1" library="rcl" library_urn="urn:adsk.eagle:library:334" deviceset="R-EU_" device="M1206" package3d_urn="urn:adsk.eagle:package:23566/1"/>
-<part name="R3" library="rcl" library_urn="urn:adsk.eagle:library:334" deviceset="R-EU_" device="M1206" package3d_urn="urn:adsk.eagle:package:23566/1"/>
+<part name="R1" library="rcl" library_urn="urn:adsk.eagle:library:334" deviceset="R-EU_" device="M1206" package3d_urn="urn:adsk.eagle:package:23566/1" value="100R"/>
+<part name="R3" library="rcl" library_urn="urn:adsk.eagle:library:334" deviceset="R-EU_" device="M1206" package3d_urn="urn:adsk.eagle:package:23566/1" value="100R"/>
 <part name="GND3" library="supply1" library_urn="urn:adsk.eagle:library:371" deviceset="GND" device=""/>
 <part name="+3V3" library="supply1" library_urn="urn:adsk.eagle:library:371" deviceset="+3V3" device=""/>
@@
 <part name="LED1" library="led" library_urn="urn:adsk.eagle:library:259" deviceset="LED" device="CHIPLED_1206" package3d_urn="urn:adsk.eagle:package:15823/2"/>
 <part name="LED3" library="led" library_urn="urn:adsk.eagle:library:259" deviceset="LED" device="CHIPLED_1206" package3d_urn="urn:adsk.eagle:package:15823/2"/>
-<part name="R2" library="pot" library_urn="urn:adsk.eagle:library:331" deviceset="TRIM_EU-" device="B64Y" package3d_urn="urn:adsk.eagle:package:22690/1"/>
+<part name="R2" library="pot" library_urn="urn:adsk.eagle:library:331" deviceset="TRIM_EU-" device="B64Y" package3d_urn="urn:adsk.eagle:package:22690/1" value="100k"/>
 <part name="+3V5" library="supply1" library_urn="urn:adsk.eagle:library:371" deviceset="+3V3" device=""/>
 <part name="GND6" library="supply1" library_urn="urn:adsk.eagle:library:371" deviceset="GND" device=""/>
@@
 <part name="SJ1" library="jumper" library_urn="urn:adsk.eagle:library:252" deviceset="SJ" device="" package3d_urn="urn:adsk.eagle:package:15471/1"/>
 <part name="SJ3" library="jumper" library_urn="urn:adsk.eagle:library:252" deviceset="SJ" device="" package3d_urn="urn:adsk.eagle:package:15471/1"/>
-<part name="SJ4" library="jumper" library_urn="urn:adsk.eagle:library:252" deviceset="SJ" device="" package3d_urn="urn:adsk.eagle:package:15471/1"/>
 <part name="SJ5" library="jumper" library_urn="urn:adsk.eagle:library:252" deviceset="SJ" device="" package3d_urn="urn:adsk.eagle:package:15471/1"/>
 <part name="U$7" library="diy-modules" deviceset="TEMP-HUM-SENSOR-DHT11" device=""/>
@@
 <part name="+3V9" library="supply1" library_urn="urn:adsk.eagle:library:371" deviceset="+3V3" device=""/>
 <part name="GND11" library="supply1" library_urn="urn:adsk.eagle:library:371" deviceset="GND" device=""/>
-<part name="GND12" library="supply1" library_urn="urn:adsk.eagle:library:371" deviceset="GND" device=""/>
 <part name="GND13" library="supply1" library_urn="urn:adsk.eagle:library:371" deviceset="GND" device=""/>
 <part name="U$8" library="Cing Library" deviceset="LEGO-1X1" device=""/>
 <part name="U$9" library="Cing Library" deviceset="LEGO-1X1" device=""/>
+<part name="R4" library="rcl" library_urn="urn:adsk.eagle:library:334" deviceset="R-EU_" device="M1206" package3d_urn="urn:adsk.eagle:package:23566/1" value="1k"/>
 </parts>
 <sheets>
@@
 <attribute name="VALUE" x="99.06" y="-25.4" size="1.778" layer="96" rot="R90"/>
 </instance>
-<instance part="SJ1" gate="1" x="144.78" y="68.58" smashed="yes">
-<attribute name="NAME" x="142.24" y="71.12" size="1.778" layer="95"/>
-<attribute name="VALUE" x="142.24" y="64.77" size="1.778" layer="96"/>
-</instance>
-<instance part="SJ3" gate="1" x="144.78" y="71.12" smashed="yes">
-<attribute name="NAME" x="142.24" y="73.66" size="1.778" layer="95"/>
-<attribute name="VALUE" x="142.24" y="67.31" size="1.778" layer="96"/>
-</instance>
-<instance part="SJ4" gate="1" x="144.78" y="60.96" smashed="yes">
-<attribute name="NAME" x="142.24" y="63.5" size="1.778" layer="95"/>
-<attribute name="VALUE" x="142.24" y="57.15" size="1.778" layer="96"/>
-</instance>
-<instance part="SJ5" gate="1" x="144.78" y="43.18" smashed="yes">
-<attribute name="NAME" x="142.24" y="45.72" size="1.778" layer="95"/>
-<attribute name="VALUE" x="142.24" y="39.37" size="1.778" layer="96"/>
+<instance part="SJ1" gate="1" x="147.32" y="68.58" smashed="yes">
+<attribute name="NAME" x="144.78" y="71.12" size="1.778" layer="95"/>
+<attribute name="VALUE" x="144.78" y="64.77" size="1.778" layer="96"/>
+</instance>
+<instance part="SJ3" gate="1" x="147.32" y="71.12" smashed="yes">
+<attribute name="NAME" x="144.78" y="73.66" size="1.778" layer="95"/>
+<attribute name="VALUE" x="144.78" y="67.31" size="1.778" layer="96"/>
+</instance>
+<instance part="SJ5" gate="1" x="147.32" y="43.18" smashed="yes">
+<attribute name="NAME" x="144.78" y="45.72" size="1.778" layer="95"/>
+<attribute name="VALUE" x="144.78" y="39.37" size="1.778" layer="96"/>
 </instance>
 <instance part="U$7" gate="G$1" x="177.8" y="83.82" smashed="yes">
@@
 <attribute name="VALUE" x="160.02" y="86.36" size="1.778" layer="96" rot="R90"/>
 </instance>
-<instance part="GND11" gate="1" x="152.4" y="66.04" smashed="yes">
-<attribute name="VALUE" x="149.86" y="63.5" size="1.778" layer="96"/>
-</instance>
-<instance part="GND12" gate="1" x="152.4" y="58.42" smashed="yes">
-<attribute name="VALUE" x="149.86" y="55.88" size="1.778" layer="96"/>
-</instance>
-<instance part="GND13" gate="1" x="152.4" y="40.64" smashed="yes">
-<attribute name="VALUE" x="149.86" y="38.1" size="1.778" layer="96"/>
+<instance part="GND11" gate="1" x="154.94" y="66.04" smashed="yes">
+<attribute name="VALUE" x="152.4" y="63.5" size="1.778" layer="96"/>
+</instance>
+<instance part="GND13" gate="1" x="154.94" y="40.64" smashed="yes">
+<attribute name="VALUE" x="152.4" y="38.1" size="1.778" layer="96"/>
 </instance>
 <instance part="U$8" gate="G$1" x="5.08" y="68.58" smashed="yes"/>
 <instance part="U$9" gate="G$1" x="-2.54" y="81.28" smashed="yes"/>
+<instance part="R4" gate="G$1" x="30.48" y="-7.62" smashed="yes">
+<attribute name="NAME" x="26.67" y="-6.1214" size="1.778" layer="95"/>
+<attribute name="VALUE" x="26.67" y="-10.922" size="1.778" layer="96"/>
+</instance>
 </instances>
 <busses>
@@
 <pinref part="SJ5" gate="1" pin="2"/>
 <pinref part="GND13" gate="1" pin="GND"/>
-<wire x1="149.86" y1="43.18" x2="152.4" y2="43.18" width="0.1524" layer="91"/>
-</segment>
-<segment>
-<pinref part="SJ4" gate="1" pin="2"/>
-<pinref part="GND12" gate="1" pin="GND"/>
-<wire x1="149.86" y1="60.96" x2="152.4" y2="60.96" width="0.1524" layer="91"/>
+<wire x1="154.94" y1="43.18" x2="152.4" y2="43.18" width="0.1524" layer="91"/>
 </segment>
 <segment>
 <pinref part="SJ1" gate="1" pin="2"/>
 <pinref part="SJ3" gate="1" pin="2"/>
-<wire x1="149.86" y1="68.58" x2="149.86" y2="71.12" width="0.1524" layer="91"/>
+<wire x1="152.4" y1="68.58" x2="152.4" y2="71.12" width="0.1524" layer="91"/>
 <pinref part="GND11" gate="1" pin="GND"/>
-<wire x1="149.86" y1="68.58" x2="152.4" y2="68.58" width="0.1524" layer="91"/>
-<junction x="149.86" y="68.58"/>
+<wire x1="152.4" y1="68.58" x2="154.94" y2="68.58" width="0.1524" layer="91"/>
+<junction x="152.4" y="68.58"/>
 </segment>
 </net>
@@
 <net name="OUTPUT" class="0">
 <segment>
-<pinref part="U$6" gate="G$1" pin="A1"/>
-<wire x1="35.56" y1="-7.62" x2="33.02" y2="-7.62" width="0.1524" layer="91"/>
-<label x="33.02" y="-7.62" size="1.778" layer="95" rot="R180" xref="yes"/>
-</segment>
-<segment>
 <pinref part="LED3" gate="G$1" pin="A"/>
 <wire x1="66.04" y1="25.4" x2="66.04" y2="27.94" width="0.1524" layer="91"/>
 <label x="66.04" y="27.94" size="1.778" layer="95" rot="R90" xref="yes"/>
+</segment>
+<segment>
+<pinref part="U$2" gate="G$1" pin="(PCINT7/ICP/OC0B/ADC7)PA7"/>
+<wire x1="142.24" y1="60.96" x2="139.7" y2="60.96" width="0.1524" layer="91"/>
+<label x="142.24" y="60.96" size="1.778" layer="95" xref="yes"/>
+</segment>
+<segment>
+<wire x1="25.4" y1="-7.62" x2="20.32" y2="-7.62" width="0.1524" layer="91"/>
+<pinref part="R4" gate="G$1" pin="1"/>
+<label x="20.32" y="-7.62" size="1.778" layer="95" rot="R180" xref="yes"/>
 </segment>
 </net>
@@
 </segment>
 </net>
-<net name="N$1" class="0">
+<net name="9" class="0">
 <segment>
 <pinref part="U$2" gate="G$1" pin="(PCINT9/XTAL2)PB1"/>
 <pinref part="SJ1" gate="1" pin="1"/>
-</segment>
-</net>
-<net name="N$3" class="0">
+<wire x1="142.24" y1="68.58" x2="139.7" y2="68.58" width="0.1524" layer="91"/>
+</segment>
+</net>
+<net name="8" class="0">
 <segment>
 <pinref part="U$2" gate="G$1" pin="(PCINT10/INT0/OC0A/CKOUT)PB2"/>
 <pinref part="SJ3" gate="1" pin="1"/>
-</segment>
-</net>
-<net name="N$4" class="0">
-<segment>
-<pinref part="U$2" gate="G$1" pin="(PCINT7/ICP/OC0B/ADC7)PA7"/>
-<pinref part="SJ4" gate="1" pin="1"/>
-</segment>
-</net>
-<net name="N$5" class="0">
+<wire x1="142.24" y1="71.12" x2="139.7" y2="71.12" width="0.1524" layer="91"/>
+</segment>
+</net>
+<net name="0" class="0">
 <segment>
 <pinref part="U$2" gate="G$1" pin="(PCINT0/AREF/ADC0)PA0"/>
 <pinref part="SJ5" gate="1" pin="1"/>
+<wire x1="142.24" y1="43.18" x2="139.7" y2="43.18" width="0.1524" layer="91"/>
 </segment>
 </net>
@@
 </segment>
 </net>
+<net name="N$1" class="0">
+<segment>
+<pinref part="U$6" gate="G$1" pin="A1"/>
+<pinref part="R4" gate="G$1" pin="2"/>
+</segment>
+</net>
