File: Hardware/Schematics/StepperModule/StepperModule.brd (EAGLE design)
At the start: 53 x 26 mm, 14 parts, among them IC1 L293D

Commit message: commit
Other:
- board size 53 x 26 mm -> 53 x 25.5 mm
- board text added: "Sponsored by JLCPCB"
Changed lines of the file:
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@@
 <board>
 <plain>
-<wire x1="-26.5" y1="-13" x2="26.5" y2="-13" width="0.0762" layer="20"/>
-<wire x1="26.5" y1="-13" x2="26.5" y2="13" width="0.0762" layer="20"/>
+<wire x1="-26.5" y1="-12.5" x2="26.5" y2="-12.5" width="0.0762" layer="20"/>
+<wire x1="26.5" y1="-12.5" x2="26.5" y2="13" width="0.0762" layer="20"/>
 <wire x1="26.5" y1="13" x2="-26.5" y2="13" width="0.0762" layer="20"/>
-<wire x1="-26.5" y1="13" x2="-26.5" y2="-13" width="0.0762" layer="20"/>
+<wire x1="-26.5" y1="13" x2="-26.5" y2="-12.5" width="0.0762" layer="20"/>
 <text x="-21" y="-12" size="1.778" layer="21" align="bottom-center">VCC mot</text>
 <text x="23.5" y="-12" size="1.778" layer="21" align="bottom-center">3.3V</text>
+<text x="0" y="10.9" size="1.778" layer="21" align="bottom-center">Sponsored by JLCPCB</text>
 </plain>
 <attributes>
@@
 <param name="mdViaViaSameLayer" value="6mil"/>
 <param name="mnLayersViaInSmd" value="2"/>
-<param name="mdCopperDimension" value="20mil"/>
+<param name="mdCopperDimension" value="10mil"/>
 <param name="mdDrill" value="6mil"/>
 <param name="mdSmdStop" value="0mil"/>
@@
 <vertex x="-28" y="14"/>
 <vertex x="29" y="14"/>
-<vertex x="29" y="-12"/>
-<vertex x="-28" y="-12"/>
+<vertex x="29" y="-14.5"/>
+<vertex x="-28" y="-14.5"/>
 </polygon>
 <wire x1="-12.7" y1="-1.27" x2="-7.62" y2="-1.27" width="1.016" layer="16"/>
@@
 <vertex x="-28" y="14"/>
 <vertex x="29" y="14"/>
-<vertex x="29" y="-12"/>
-<vertex x="-28" y="-12"/>
+<vertex x="29" y="-14"/>
+<vertex x="-28" y="-14"/>
 </polygon>
 <contactref element="LED1" pad="C"/>

Commit message: gerber update
Other:
- outline, holes or cut-outs redrawn
- board text added: "Stepper Module for robot Cing"
- board text removed: "Sponsored by JLCPCB"
Changed lines of the file:
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@@
 <?xml version="1.0" encoding="utf-8"?>
 <!DOCTYPE eagle SYSTEM "eagle.dtd">
-<eagle version="9.2.2">
+<eagle version="9.4.0">
 <drawing>
 <settings>
@@
 <board>
 <plain>
-<wire x1="-26.5" y1="-12.5" x2="26.5" y2="-12.5" width="0.0762" layer="20"/>
-<wire x1="26.5" y1="-12.5" x2="26.5" y2="13" width="0.0762" layer="20"/>
-<wire x1="26.5" y1="13" x2="-26.5" y2="13" width="0.0762" layer="20"/>
-<wire x1="-26.5" y1="13" x2="-26.5" y2="-12.5" width="0.0762" layer="20"/>
+<wire x1="26.5" y1="-11.5" x2="26.5" y2="12" width="0.0762" layer="20"/>
+<wire x1="25.5" y1="13" x2="-25.5" y2="13" width="0.0762" layer="20"/>
 <text x="-21" y="-12" size="1.778" layer="21" align="bottom-center">VCC mot</text>
 <text x="23.5" y="-12" size="1.778" layer="21" align="bottom-center">3.3V</text>
-<text x="0" y="10.9" size="1.778" layer="21" align="bottom-center">Sponsored by JLCPCB</text>
+<text x="0" y="10.9" size="1.778" layer="21" align="bottom-center">Stepper Module for robot Cing</text>
+<wire x1="-26.5" y1="12" x2="-26.5" y2="-11.5" width="0.0762" layer="20"/>
+<wire x1="-25.5" y1="-12.5" x2="-26.5" y2="-11.5" width="0.0762" layer="20" curve="-90"/>
+<wire x1="26.5" y1="-11.5" x2="25.5" y2="-12.5" width="0.0762" layer="20" curve="-90"/>
+<wire x1="25.5" y1="13" x2="26.5" y2="12" width="0.0762" layer="20" curve="-90"/>
+<wire x1="-26.5" y1="12" x2="-25.5" y2="13" width="0.0762" layer="20" curve="-90"/>
+<wire x1="-25.5" y1="-12.5" x2="25.5" y2="-12.5" width="0.0762" layer="20"/>
 </plain>
 <attributes>
