File: Hardware/Schematics/Cing_MainBoard/Cing_MainBoard.brd (EAGLE design)
At the start: 100 x 100 mm, 169 parts, among them IC1 L293D, IC2 LM2576S, IC3 FT232RL, IC5 BME280, Q1 16mhz, Q2 BSS138, Q3 BSS138, Q4 BSS138, Q5 BSS138, Q6 NP2301AMR-G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

Commit message: commit
Parts:
- removed R36: 10k, rcl:R1206
- removed U$9: LM1117-5V, Cing Library:LM1117
- added R44: 10k, rcl:R1206
- R49: value 7k5 -> 12K
- R7: value 1k -> 10k
- R9: value 12k -> 10k
Connections:
- removed net VDD: U$13.8, U$14.1, U$9.2, U$9.TAB
- net +3V3: no longer R36.1
- net +5V: now also R44.1
- net A0: now also SW7.COM1; no longer SW7.CH1B
- net A0H: now also SW7.CH1B; no longer SW7.COM1
- net BAT+: no longer U$9.3
- net BAT-: now also ON.C, R6.1
- net GND: no longer ON.C, R6.1, U$9.1
- net RESET: no longer R36.2
- net VCC_SERVO: now also R44.2, U$13.8, U$14.1
Routing:
- net VCC_SERVO: track 121.3 -> 349.8 mm, vias 2 -> 9
- net VDD: track 163.1 -> 0.00 mm, vias 6 -> 0
- net GND: track 896.0 -> 865.0 mm
- net BAT-: track 93.6 -> 119.8 mm, vias 1 -> 2
- net BAT+: track 298.8 -> 287.3 mm, vias 12 -> 9
- net RESET: track 194.0 -> 185.9 mm, vias 10 -> 9
- net +5V: track 28.1 -> 35.4 mm
- net +3V3: track 674.2 -> 671.7 mm
- net A6: track 32.9 -> 35.1 mm
- net A0: track 78.1 -> 76.2 mm

Commit message: c
Parts:
- moved R29 1.92 mm to (32.2, 41.2)
- turned JP4 to 0 degrees
Routing:
- net GND: track 865.0 -> 853.4 mm
- net D6: track 119.5 -> 126.5 mm, vias 3 -> 5
- net +3V3: track 671.7 -> 668.5 mm
- net N$66: track 10.0 -> 11.1 mm

Commit message: commit
Routing:
- net BAT-: track 119.8 -> 117.8 mm
Changed lines of the file:
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@@
 <wire x1="3.1" y1="-48.8" x2="25.146" y2="-48.8" width="0.508" layer="16"/>
 <contactref element="R6" pad="1"/>
-<wire x1="20.7" y1="-36.3" x2="20" y2="-35.6" width="0.4064" layer="16"/>
 <via x="17" y="-35.6" extent="1-16" drill="0.35"/>
-<wire x1="21.0838" y1="-37.04605" x2="21.0838" y2="-37.65395" width="0.4064" layer="16"/>
-<wire x1="21.0838" y1="-37.65395" x2="20.65395" y2="-38.0838" width="0.4064" layer="16"/>
+<wire x1="20.65395" y1="-38.0838" x2="21.0838" y2="-37.65395" width="0.4064" layer="16"/>
 <wire x1="20.65395" y1="-38.0838" x2="18.00985" y2="-38.0838" width="0.4064" layer="16"/>
 <wire x1="18.00985" y1="-38.0838" x2="17.1532" y2="-37.22715" width="0.4064" layer="16"/>
-<wire x1="20" y1="-35.6" x2="20" y2="-35.96225" width="0.4064" layer="16"/>
-<wire x1="20" y1="-35.96225" x2="21.0838" y2="-37.04605" width="0.4064" layer="16"/>
 <wire x1="17.1532" y1="-35.7532" x2="17" y2="-35.6" width="0.4064" layer="16"/>
 <wire x1="17.1532" y1="-37.22715" x2="17.1532" y2="-35.7532" width="0.4064" layer="16"/>
@@
 <wire x1="16.34879375" y1="-26.4224" x2="17" y2="-27.07360625" width="0.4064" layer="1"/>
 <wire x1="17" y1="-27.07360625" x2="17" y2="-35.6" width="0.4064" layer="1"/>
+<wire x1="21.0838" y1="-36.6838" x2="20.7" y2="-36.3" width="0.4064" layer="16"/>
+<wire x1="21.0838" y1="-37.65395" x2="21.0838" y2="-36.6838" width="0.4064" layer="16"/>
 </signal>
 <signal name="N$3">

Commit message: commit
Parts:
- R41: value 2 -> 2R
Changed lines of the file:
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@@
 </element>
 <element name="U$13" library="bt_adc" package="MSOP10_0.5" value="ADS1015IDGT" x="-21.1" y="-41.4" smashed="yes" rot="MR180"/>
-<element name="R41" library="rcl" library_urn="urn:adsk.eagle:library:334" package="R2512" package3d_urn="urn:adsk.eagle:package:23545/2" value="2" x="-15.3" y="-32.5" smashed="yes" rot="MR180">
+<element name="R41" library="rcl" library_urn="urn:adsk.eagle:library:334" package="R2512" package3d_urn="urn:adsk.eagle:package:23545/2" value="2R" x="-15.3" y="-32.5" smashed="yes" rot="MR180">
 <attribute name="SPICEPREFIX" value="R" x="-15.3" y="-32.5" size="1.778" layer="28" rot="MR180" display="off"/>
 </element>

Commit message: PCB version 3.0.1
Parts:
- removed C4, C9: 100uf, rcl:E3,5-8
- added JP23: (no value), pinhead:1X02
- added U$24, U$9: POLULU_MOTOR, Cing Library:POLULU_MOTOR
- moved S2 77.8 mm to (37.3, -17.6), turned to 270 degrees
- moved JP3 31.1 mm to (-45.8, 29.0)
- moved JP2 27.6 mm to (-45.8, 25.8)
- moved IC2 18.0 mm to (-17.0, 26.5)
- moved L2 16.3 mm to (-6.50, 42.8), turned to 180 degrees
- moved D1 16.2 mm to (-42.8, 20.2)
- moved WS2812 15.0 mm to (45.0, -36.6), turned to 180 degrees
- moved C17 14.1 mm to (-27.0, 27.7), turned to 45 degrees
- moved L1 12.7 mm to (-12.2, 43.0), turned to 180 degrees
- moved C20 8.22 mm to (-4.59, 33.2), turned to 90 degrees
- moved U$11 8.17 mm to (-5.70, -44.3)
- moved R32 8.05 mm to (30.7, -39.5), turned to 90 degrees
- moved BT1 6.24 mm to (6.20, -44.7)
- moved U$7 6.24 mm to (6.20, -44.7)
- moved U$13 6.07 mm to (-15.4, -43.5)
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Connections:
- net +3V3: no longer C4.+
- net BAT+: no longer C9.+
- net GND: no longer C4.-, C9.-
- net MOT_A+: now also U$24.+
- net MOT_A-: now also U$24.-
- net MOT_B+: now also U$9.+
- net MOT_B-: now also U$9.-
- net SCL: now also JP23.2
- net SDA: now also JP23.1
Routing:
- net MOT_B-: track 12.8 -> 66.5 mm, vias 0 -> 2
- net MOT_A+: track 24.3 -> 71.5 mm, vias 0 -> 2
- net N$21: track 15.1 -> 62.3 mm, vias 0 -> 4
- net BAT+: track 287.3 -> 322.0 mm
- net MOT_A-: track 15.0 -> 46.0 mm, vias 0 -> 1
- net N$2: track 86.2 -> 116.1 mm
- net MOT_B+: track 23.2 -> 52.1 mm
- net IN_A2: track 112.8 -> 84.3 mm
- net IN_A1: track 116.9 -> 92.3 mm, vias 6 -> 4
- net SDA: track 225.4 -> 247.2 mm, vias 7 -> 9
- net VCC_SERVO: track 349.8 -> 370.9 mm
- net N$44: track 16.4 -> 35.0 mm
- net +3V3: track 668.5 -> 650.3 mm
- net SCL: track 223.0 -> 240.6 mm, vias 7 -> 8
- net IRFU: track 100.4 -> 84.6 mm
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
Commit message: Board version 3.1
Parts:
- VERSION: value 3.0 -> 3.1
Other:
- board text added: "A"
- board text added: "B"
- board text added: "Created by RobotCing Team: Veronika Nemjová Stanley Jochman Designed in Slovakia"
- board text removed: "Created by RobotCing Team: Veronika Nemjová Stanley Jochman Designed in Slovakia Sponsored by PCBWay"
Changed lines of the file:
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@@
 Stanley Jochman
 Designed in Slovakia
-Sponsored by PCBWay</text>
+</text>
 <text x="-46.702" y="22.21" size="1.27" layer="21">ON</text>
 <text x="-47.002" y="12.21" size="1.27" layer="21">OFF</text>
@@
 <text x="0.945" y="28.848" size="1.778" layer="21">Header 3</text>
 <text x="-10.755" y="28.348" size="1.778" layer="21">BT</text>
+<text x="-34.8" y="-43.7" size="3.81" layer="21" rot="R90" align="center">B</text>
+<text x="-34.8" y="43.7" size="3.81" layer="21" rot="R90" align="center">A</text>
 </plain>
 <attributes>
@@
 <element name="R15" library="rcl" library_urn="urn:adsk.eagle:library:334" package="R1206" package3d_urn="urn:adsk.eagle:package:23540/2" value="10k" x="-31.5" y="6.65" smashed="yes" rot="R180">
 <attribute name="SPICEPREFIX" value="R" x="-31.5" y="6.65" size="1.778" layer="27" rot="R180" display="off"/>
-<attribute name="VALUE" x="-26.166" y="7.285" size="1.27" layer="27" rot="R180"/>
 </element>
 <element name="R16" library="rcl" library_urn="urn:adsk.eagle:library:334" package="R1206" package3d_urn="urn:adsk.eagle:package:23540/2" value="100" x="31" y="-10" smashed="yes" rot="R270">
@@
 <attribute name="OC_FARNELL" value="176432" x="41.5" y="-27" size="1.778" layer="27" display="off"/>
 <attribute name="OC_NEWARK" value="36M3542" x="41.5" y="-27" size="1.778" layer="27" display="off"/>
-<attribute name="VALUE" x="37.436" y="-32.715" size="2.1844" layer="21" ratio="10"/>
+<attribute name="VALUE" x="38.636" y="-33.015" size="1.6764" layer="21" ratio="10"/>
 </element>
 <element name="U$1" library="Cing Library" package="PROCESSOR-SOCKET_PCB" package3d_urn="urn:adsk.eagle:package:10154714/1" value="PROCESSOR-SOCKET_PCB" x="0" y="0" smashed="yes"/>
@@
 <attribute name="NAME" x="17.713" y="-28.746" size="1.27" layer="27" rot="R90"/>
 </element>
-<element name="VERSION" library="Cing Library" package="VERSION" package3d_urn="urn:adsk.eagle:package:10154717/1" value="3.0" x="49.5" y="0" smashed="yes" rot="R90">
+<element name="VERSION" library="Cing Library" package="VERSION" package3d_urn="urn:adsk.eagle:package:10154717/1" value="3.1" x="49.5" y="0" smashed="yes" rot="R90">
 <attribute name="VALUE" x="46.5" y="6.84" size="2.54" layer="21" rot="R90" align="center"/>
 </element>
@@
 <element name="C14" library="rcl" library_urn="urn:adsk.eagle:library:334" package="C1206" package3d_urn="urn:adsk.eagle:package:23618/2" value="22uf" x="-27" y="10.3" smashed="yes">
 <attribute name="SPICEPREFIX" value="C" x="-27" y="10.3" size="1.778" layer="27" display="off"/>
-<attribute name="VALUE" x="-28.27" y="7.76" size="1.27" layer="27"/>
 </element>
 <element name="C15" library="rcl" library_urn="urn:adsk.eagle:library:334" package="C1206" package3d_urn="urn:adsk.eagle:package:23618/2" value="22uf" x="-7.5584" y="20.9744" smashed="yes" rot="R270">
@@
 </element>
 <element name="JP23" library="pinhead" library_urn="urn:adsk.eagle:library:325" package="1X02" package3d_urn="urn:adsk.eagle:package:22435/2" value="" x="-18.85" y="0" smashed="yes" rot="R90">
-<attribute name="NAME" x="-20.6788" y="-2.6162" size="1.27" layer="25" ratio="10" rot="R90"/>
 <attribute name="VALUE" x="-15.675" y="-2.54" size="1.27" layer="27" rot="R90"/>
 </element>
