File: Hardware/Schematics/Cing_MainBoard/Cing_MainBoard.sch (EAGLE design)
At the start: 169 parts, among them IC1 L293D, IC2 LM2576S, IC3 FT232RL, IC5 BME280, Q1 16mhz, Q2 BSS138, Q3 BSS138, Q4 BSS138, Q5 BSS138, Q6 NP2301AMR-G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

Commit message: commit
Parts:
- removed R36: 10k, rcl:R-EU_R1206
- removed U$9: LM1117-5V, Cing Library:LM1117
- added R44: 10k, rcl:R-EU_R1206
- R49: value 7k5 -> 12K
- R7: value 1k -> 10k
- R9: value 12k -> 10k
Connections:
- removed net VDD: U$13.VDD, U$14.VIN, U$9.OUT, U$9.VO
- net +3V3: no longer R36.1
- net +5V: now also R44.1
- net A0: now also SW7.COM1; no longer SW7.CH1B
- net A0H: now also SW7.CH1B; no longer SW7.COM1
- net BAT+: no longer U$9.VI
- net BAT-: now also ON.C, R6.1
- net GND: no longer ON.C, R6.1, U$9.GND
- net RESET: no longer R36.2
- net VCC_SERVO: now also R44.2, U$13.VDD, U$14.VIN

Commit message: commit
Parts:
- R41: value 2 -> 2R
Changed lines of the file:
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@@
 <part name="U$13" library="bt_adc" deviceset="ADS1015" device="IDGT"/>
 <part name="GND46" library="supply1" library_urn="urn:adsk.eagle:library:371" deviceset="GND" device=""/>
-<part name="R41" library="rcl" library_urn="urn:adsk.eagle:library:334" deviceset="R-EU_" device="R2512" package3d_urn="urn:adsk.eagle:package:23545/2" value="2"/>
+<part name="R41" library="rcl" library_urn="urn:adsk.eagle:library:334" deviceset="R-EU_" device="R2512" package3d_urn="urn:adsk.eagle:package:23545/2" value="2R"/>
 <part name="IC2" library="lm2576" deviceset="LM2576" device="S"/>
 <part name="C17" library="rcl" library_urn="urn:adsk.eagle:library:334" deviceset="CPOL-EU" device="E3.5-8" package3d_urn="urn:adsk.eagle:package:23360/2"/>

Commit message: PCB version 3.0.1
Parts:
- removed C4, C9: 100uf, rcl:CPOL-EUE3.5-8
- added JP23: (no value), pinhead:PINHD-1X2
- added U$24, U$9: POLULU_MOTOR, Cing Library:POLULU_MOTOR
Connections:
- net +3V3: no longer C4.+
- net BAT+: no longer C9.+
- net GND: no longer C4.-, C9.-
- net MOT_A+: now also U$24.+
- net MOT_A-: now also U$24.-
- net MOT_B+: now also U$9.+
- net MOT_B-: now also U$9.-
- net SCL: now also JP23.2
- net SDA: now also JP23.1

Commit message: Board version 3.1
Parts:
- VERSION: value 3.0 -> 3.1
Changed lines of the file:
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@@
 <part name="R6" library="rcl" library_urn="urn:adsk.eagle:library:334" deviceset="R-EU_" device="R1206" package3d_urn="urn:adsk.eagle:package:23540/2" value="100"/>
 <part name="REVERSE" library="led" library_urn="urn:adsk.eagle:library:259" deviceset="LED" device="SMT1206" package3d_urn="urn:adsk.eagle:package:15796/2" value="RED"/>
-<part name="VERSION" library="Cing Library" deviceset="VERSION" device="" package3d_urn="urn:adsk.eagle:package:10154717/1" value="3.0"/>
+<part name="VERSION" library="Cing Library" deviceset="VERSION" device="" package3d_urn="urn:adsk.eagle:package:10154717/1" value="3.1"/>
 <part name="SW1" library="Cing Library" deviceset="USB_SWITCH" device="" package3d_urn="urn:adsk.eagle:package:10154743/1"/>
 <part name="U1" library="Cing Library" deviceset="MICRO_USB" device="&quot;&quot;" package3d_urn="urn:adsk.eagle:package:10154724/1"/>
