File: Hardware/Schematics/MainBoard/Cing_MainBoard.brd (EAGLE design)
At the start: 100 x 100 mm, 180 parts, among them IC1 L293D, IC2 LM2576S, IC3 FT232RL, IC5 BME280, Q1 16mhz, Q2 BSS138, Q3 BSS138, Q4 BSS138, Q5 BSS138, Q6 NP2301AMR-G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

Commit message: adding CH330N
Parts:
- added C28, C29: 100n, rcl:C1206
- added U4: CH330N, Cing Library:SOIC-8N
Connections:
- net +3V3: now also C28.1, C29.2, U4.5, U4.8
- net D+: now also U4.1
- net D-: now also U4.2
- net GND: now also C28.2, C29.1, U1.ID1, U4.3
- net RXD: now also U4.6
- net TXD: now also U4.7
Routing:
- net +3V3: track 642.1 -> 682.6 mm
- net D+: track 19.4 -> 39.4 mm, vias 0 -> 3
- net RXD: track 103.3 -> 120.7 mm
- net TXD: track 111.5 -> 127.9 mm, vias 5 -> 6
- net GND: track 874.9 -> 889.0 mm, vias 48 -> 50
- net D-: track 23.3 -> 30.2 mm, vias 2 -> 3
- net SCL: track 239.5 -> 237.9 mm
- net N$39: track 39.0 -> 39.8 mm
- net RESET: track 209.7 -> 210.3 mm
- net N$65: track 9.99 -> 10.6 mm
- net N$8: track 20.1 -> 19.6 mm

Commit message: commit
Parts:
- added C30, C31: 100n, rcl:C1206
- added IC4: BMP280, bosch-bmp280:BMP280
Connections:
- net +3V3: now also C30.2, C31.2, IC4.2, IC4.5, IC4.6, IC4.8
- net GND: now also C30.1, C31.1, IC4.1, IC4.7
- net SCL: now also IC4.4
- net SDA: now also IC4.3
Routing:
- net GND: track 889.0 -> 925.5 mm, vias 50 -> 52
- net +3V3: track 682.6 -> 696.6 mm, vias 40 -> 41
- net SCL: track 237.9 -> 245.6 mm
- net SDA: track 245.0 -> 252.0 mm, vias 9 -> 10
- net RESET: track 210.3 -> 209.6 mm
- net A0: track 77.3 -> 77.9 mm

Commit message: commit
Parts:
- moved C15 5.70 mm to (-12.1, 24.5)
- moved U$23 5.31 mm to (-8.80, 26.9), turned to 90 degrees
- moved C17 2.14 mm to (-20.5, 32.1)
- moved C23 1.43 mm to (-26.2, 27.5)
Routing:
- net BAT+: track 310.7 -> 287.2 mm
- net +3V3: track 696.6 -> 712.2 mm
- net GND: track 925.5 -> 928.4 mm, vias 52 -> 53
- net D2: track 50.3 -> 51.9 mm
- net N$11: track 102.0 -> 103.5 mm
- net HD_A6: track 73.1 -> 71.9 mm
- net VCC_MOT: track 53.9 -> 55.0 mm
- net D5: track 88.2 -> 87.2 mm
Other:
- board text added: "Bluetooth"
- board text added: "JP"

Commit message: commit
Parts:
- moved R40 13.1 mm to (-32.9, -27.7), turned to 270 degrees
- moved C10 4.08 mm to (-17.3, -48.8)
- moved WS2812 0.90 mm to (45.0, -35.7)
Routing:
- net GND: track 928.4 -> 950.9 mm
- net +3V3: track 712.2 -> 704.1 mm
- net VUSB: track 33.0 -> 34.1 mm
- net SCL: track 245.6 -> 244.8 mm
- net SCK: track 145.6 -> 145.9 mm, vias 9 -> 11

Commit message: adding minor fixes
Parts:
- R22, R6: value 100 -> R100
- R41: device rcl:R2512 -> rcl:R1206
- moved C20 0.71 mm to (-5.29, 33.1)
Routing:
- net +3V3: track 704.1 -> 701.1 mm
- net VCC_SERVO: track 521.1 -> 522.8 mm
- net CUR-SENSE: track 47.5 -> 48.4 mm
- net GND: track 950.9 -> 951.6 mm
- net BAT+: track 287.2 -> 286.7 mm

Commit message: minor changes
Parts:
- moved L1 1.91 mm to (-14.1, 42.8)
- moved U$22 1.22 mm to (18.3, 44.8)
Routing:
- net N$44: track 33.5 -> 32.5 mm
- net BAT+: track 286.7 -> 285.9 mm
Other:
- board text added: "Created by RobotCing Team: Stanley Jochman Designed in Slovakia http://robotcing.sk Supported by Leaf"
- board text removed: "Created by RobotCing Team: Veronika Nemjová Stanley Jochman Designed in Slovakia Supported by Leaf"
Changed lines of the file:
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@@
 <layer number="25" name="tNames" color="7" fill="1" visible="yes" active="yes"/>
 <layer number="26" name="bNames" color="7" fill="1" visible="yes" active="yes"/>
-<layer number="27" name="tValues" color="7" fill="1" visible="yes" active="yes"/>
+<layer number="27" name="tValues" color="7" fill="1" visible="no" active="yes"/>
 <layer number="28" name="bValues" color="7" fill="1" visible="no" active="yes"/>
 <layer number="29" name="tStop" color="7" fill="3" visible="no" active="yes"/>
@@
 <wire x1="45" y1="50" x2="50" y2="45" width="0.0762" layer="20" curve="-90"/>
 <wire x1="-50" y1="45" x2="-45" y2="50" width="0.0762" layer="20" curve="-90"/>
-<text x="-4.9006" y="37.4256" size="1.6764" layer="21">Created by RobotCing Team:
-Veronika Nemjová
+<text x="-6.7006" y="37.8256" size="1.6764" layer="21">Created by RobotCing Team:
 Stanley Jochman
 Designed in Slovakia
+http://robotcing.sk
 Supported by Leaf</text>
 <text x="-46.702" y="22.21" size="1.27" layer="21">ON</text>
@@
 </element>
 <element name="U$6" library="Cing Library" library_urn="urn:adsk.eagle:library:10154637" package="BATTERY_CONECTOR_D" package3d_urn="urn:adsk.eagle:package:10154722/1" override_package3d_urn="urn:adsk.eagle:package:11838348/2" override_package_urn="urn:adsk.eagle:footprint:10154693/1" value="BATTERY_CONECTOR_D" x="-34.666" y="15.431" smashed="yes" rot="R90"/>
-<element name="U$22" library="Cing Library" library_urn="urn:adsk.eagle:library:10154637" package="OSHW_5MM" package3d_urn="urn:adsk.eagle:package:10154747/1" value="OPENSOURCE" x="17.3188" y="44.1198" smashed="yes"/>
+<element name="U$22" library="Cing Library" library_urn="urn:adsk.eagle:library:10154637" package="OSHW_5MM" package3d_urn="urn:adsk.eagle:package:10154747/1" value="OPENSOURCE" x="18.3188" y="44.8198" smashed="yes"/>
 <element name="R21" library="LDR" package="LDR_OFFBOARD" override_package3d_urn="urn:adsk.eagle:package:11838426/2" override_package_urn="urn:adsk.eagle:footprint:11838427/1" value="PHOTOCELL1" x="36.7" y="-43" smashed="yes" rot="R270"/>
 <element name="R23" library="LDR" package="LDR_OFFBOARD" override_package3d_urn="urn:adsk.eagle:package:11838375/2" override_package_urn="urn:adsk.eagle:footprint:11838376/1" value="PHOTOCELL1" x="36.7" y="43" smashed="yes" rot="R90"/>
@@
 </element>
 <element name="U$5" library="MT3608" package="SOT23-6" override_package3d_urn="urn:adsk.eagle:package:11833700/2" override_package_urn="urn:adsk.eagle:footprint:11833701/1" value="MT3608SOT23-6" x="-23.2" y="18.9" smashed="yes" rot="R90"/>
-<element name="L1" library="inductors" library_urn="urn:adsk.eagle:library:243" package="DR125" package3d_urn="urn:adsk.eagle:package:15121/1" override_package3d_urn="urn:adsk.eagle:package:11834588/2" override_package_urn="urn:adsk.eagle:footprint:15035/1" value="DR125" x="-12.2" y="43" smashed="yes" rot="R180">
-<attribute name="NAME" x="-9.70000625" y="40.000003125" size="1.27" layer="25" rot="R180"/>
-<attribute name="SPICEPREFIX" value="L" x="-12.2" y="43" size="1.778" layer="27" rot="R180" display="off"/>
+<element name="L1" library="inductors" library_urn="urn:adsk.eagle:library:243" package="DR125" package3d_urn="urn:adsk.eagle:package:15121/1" override_package3d_urn="urn:adsk.eagle:package:11834588/2" override_package_urn="urn:adsk.eagle:footprint:15035/1" value="DR125" x="-14.1" y="42.8" smashed="yes" rot="R180">
+<attribute name="NAME" x="-11.60000625" y="39.800003125" size="1.27" layer="25" rot="R180"/>
+<attribute name="SPICEPREFIX" value="L" x="-14.1" y="42.8" size="1.778" layer="27" rot="R180" display="off"/>
 </element>
 <element name="D3" library="adafruit" library_urn="urn:adsk.eagle:library:420" package="SMADIODE" package3d_urn="urn:adsk.eagle:package:6240747/1" override_package3d_urn="urn:adsk.eagle:package:11834402/2" override_package_urn="urn:adsk.eagle:footprint:6240101/1" value="" x="-26" y="13.6" smashed="yes">
@@
 <wire x1="21.28" y1="-26.0162" x2="21.3962" y2="-25.9" width="0.8128" layer="16"/>
 <wire x1="21.3962" y1="-25.9" x2="35.56" y2="-25.9" width="0.8128" layer="16"/>
-<wire x1="-10.1128" y1="36.99378125" x2="-10.1128" y2="27.82" width="0.8128" layer="1"/>
 <wire x1="-10.1128" y1="27.82" x2="-12.0584" y2="25.8744" width="0.8128" layer="1"/>
 <wire x1="-12.0584" y1="25.8744" x2="-13.5996" y2="24.3332" width="0.8128" layer="1"/>
@@
 <wire x1="16.9" y1="46.7" x2="16.9" y2="33.3" width="0.8128" layer="1"/>
 <wire x1="16.9" y1="46.7" x2="15.1" y2="48.5" width="0.8128" layer="1"/>
-<wire x1="15.1" y1="48.5" x2="-7.2" y2="48.5" width="0.8128" layer="1"/>
-<wire x1="-7.2" y1="48.5" x2="-39.17" y2="48.5" width="0.8128" layer="1"/>
-<wire x1="-7.225" y1="43" x2="-7.225" y2="48.475" width="0.8128" layer="1"/>
-<wire x1="-7.225" y1="48.475" x2="-7.2" y2="48.5" width="0.8128" layer="1"/>
-<wire x1="-7.225" y1="43" x2="-7.225" y2="39.88158125" width="0.8128" layer="1"/>
-<wire x1="-7.225" y1="39.88158125" x2="-10.1128" y2="36.99378125" width="0.8128" layer="1"/>
+<wire x1="15.1" y1="48.5" x2="-9" y2="48.5" width="0.8128" layer="1"/>
+<wire x1="-9" y1="48.5" x2="-39.17" y2="48.5" width="0.8128" layer="1"/>
+<wire x1="-9.125" y1="42.8" x2="-9.125" y2="48.375" width="0.8128" layer="1"/>
+<wire x1="-9.125" y1="48.375" x2="-9" y2="48.5" width="0.8128" layer="1"/>
+<wire x1="-9.125" y1="42.8" x2="-10.1128" y2="41.8122" width="0.8128" layer="1"/>
+<wire x1="-10.1128" y1="41.8122" x2="-10.1128" y2="27.82" width="0.8128" layer="1"/>
 <wire x1="25.11050625" y1="31.6593875" x2="18.5406125" y2="31.6593875" width="0.8128" layer="1"/>
 <wire x1="18.5406125" y1="31.6593875" x2="16.9" y2="33.3" width="0.8128" layer="1"/>
@@
 <wire x1="-23.2" y1="18.32608125" x2="-23.6352" y2="17.89088125" width="0.6096" layer="1"/>
 <wire x1="-23.9747" y1="22.2253" x2="-23.9747" y2="20.57561875" width="0.6096" layer="1"/>
-<wire x1="-19.375" y1="25.475" x2="-17.175" y2="27.675" width="0.6096" layer="1"/>
-<wire x1="-17.175" y1="27.675" x2="-17.175" y2="43" width="0.6096" layer="1"/>
+<wire x1="-19.375" y1="25.475" x2="-19.075" y2="25.775" width="0.6096" layer="1"/>
+<wire x1="-19.075" y1="25.775" x2="-19.075" y2="42.8" width="0.6096" layer="1"/>
 <wire x1="-20.725" y1="25.475" x2="-19.375" y2="25.475" width="0.6096" layer="1"/>
 <wire x1="-23.9747" y1="22.2253" x2="-20.725" y2="25.475" width="0.6096" layer="1"/>

Commit message: minor changes
Parts:
- VERSION: value 4.0 -> 4.1
Changed lines of the file:
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@@
 <attribute name="NAME" x="15.813" y="-26.546" size="1.27" layer="21" rot="R90"/>
 </element>
-<element name="VERSION" library="Cing Library" library_urn="urn:adsk.eagle:library:10154637" package="VERSION" package3d_urn="urn:adsk.eagle:package:10154717/1" value="4.0" x="49.5" y="0" smashed="yes" rot="R90">
+<element name="VERSION" library="Cing Library" library_urn="urn:adsk.eagle:library:10154637" package="VERSION" package3d_urn="urn:adsk.eagle:package:10154717/1" value="4.1" x="49.5" y="0" smashed="yes" rot="R90">
 <attribute name="VALUE" x="46.5" y="6.84" size="2.54" layer="21" rot="R90" align="center"/>
 </element>
