File: Hardware/Schematics/MainBoard/Cing_MainBoard.brd (EAGLE design)
At the start: 100 x 100 mm, 186 parts, among them IC1 L293D, IC2 LM2576S, IC3 FT232RL, IC4 BMP280, IC5 BME280, Q1 16mhz, Q2 BSS138, Q3 BSS138, Q4 BSS138, Q5 BSS138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

Commit message: 4.1 board
Parts:
- moved C21 13.7 mm to (-6.10, 2.20), flipped to the bottom
- moved JP4 0.30 mm to (30.0, 47.0)
- flipped U3 to the bottom
Connections:
- net +3V3: no longer WS2812.1
- net VCC_SERVO: now also WS2812.1
Routing:
- net VCC_SERVO: track 522.8 -> 617.1 mm
- net +3V3: track 701.1 -> 684.8 mm, vias 41 -> 43
- net GND: track 951.6 -> 943.8 mm
- net SCL: track 244.8 -> 237.6 mm
- net SDA: track 252.0 -> 249.7 mm
- net D4: track 107.4 -> 109.4 mm
- net BAT+: track 285.9 -> 287.7 mm
- net BAT-: track 133.4 -> 131.7 mm
- net CUR-SENSE: track 48.4 -> 47.3 mm
- net RESET: track 209.6 -> 209.1 mm
Other:
- board text added: "3"
- board text added: "4"
- board text added: "BTN"
- board text added: "Header"
- board text added: "LDR"

Commit message: fixing some bugs
Parts:
- R10, R20: value 1k -> 4k7
Changed lines of the file:
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@@
 <element name="TXD1" library="led" library_urn="urn:adsk.eagle:library:259" package="1206" package3d_urn="urn:adsk.eagle:package:15796/2" value="LightSensor 1" x="25" y="4" smashed="yes" rot="R90"/>
 <element name="TXD2" library="led" library_urn="urn:adsk.eagle:library:259" package="1206" package3d_urn="urn:adsk.eagle:package:15796/2" value="LightSensor 2" x="25" y="-4" smashed="yes" rot="R270"/>
-<element name="R10" library="rcl" library_urn="urn:adsk.eagle:library:334" package="R1206" package3d_urn="urn:adsk.eagle:package:23540/2" override_package3d_urn="urn:adsk.eagle:package:11835284/2" override_package_urn="urn:adsk.eagle:footprint:23047/1" value="1k" x="18.5" y="2.5" smashed="yes" rot="R180">
+<element name="R10" library="rcl" library_urn="urn:adsk.eagle:library:334" package="R1206" package3d_urn="urn:adsk.eagle:package:23540/2" override_package3d_urn="urn:adsk.eagle:package:11835284/2" override_package_urn="urn:adsk.eagle:footprint:23047/1" value="4k7" x="18.5" y="2.5" smashed="yes" rot="R180">
 <attribute name="SPICEPREFIX" value="R" x="18.5" y="2.5" size="1.778" layer="27" rot="R180" display="off"/>
 <attribute name="VALUE" x="19.77" y="5.04" size="1.27" layer="27" rot="R180"/>
 </element>
-<element name="R20" library="rcl" library_urn="urn:adsk.eagle:library:334" package="R1206" package3d_urn="urn:adsk.eagle:package:23540/2" override_package3d_urn="urn:adsk.eagle:package:11835283/2" override_package_urn="urn:adsk.eagle:footprint:23047/1" value="1k" x="18.5" y="-2.5" smashed="yes" rot="R180">
+<element name="R20" library="rcl" library_urn="urn:adsk.eagle:library:334" package="R1206" package3d_urn="urn:adsk.eagle:package:23540/2" override_package3d_urn="urn:adsk.eagle:package:11835283/2" override_package_urn="urn:adsk.eagle:footprint:23047/1" value="4k7" x="18.5" y="-2.5" smashed="yes" rot="R180">
 <attribute name="SPICEPREFIX" value="R" x="18.5" y="-2.5" size="1.778" layer="27" rot="R180" display="off"/>
 <attribute name="VALUE" x="19.77" y="0.04" size="1.27" layer="27" rot="R180"/>

Commit message: gerber update
Parts:
- R44: value 10k -> 100R
- moved R38 19.1 mm to (-2.70, -15.6), turned to 180 degrees
- moved U$14 4.50 mm to (25.0, 0.00)
- moved TSOP4838 4.10 mm to (32.1, 0.00)
- moved R19 3.01 mm to (20.9, 7.07), turned to 0 degrees
- moved JP23 2.54 mm to (-16.3, 0.00)
- moved U$22 2.51 mm to (16.1, 43.6)
- moved C19 1.25 mm to (-2.86, 28.8)
- moved R48 1.10 mm to (21.7, -25.7)
- moved C24 0.98 mm to (-30.3, 28.0)
- moved U$8 0.90 mm to (24.0, -29.9)
- moved C20 0.71 mm to (-5.99, 33.0)
- moved Q2 0.10 mm to (8.50, -24.4)
Routing:
- net GND: track 943.8 -> 920.2 mm
- net SCL: track 237.6 -> 221.9 mm
- net SDA: track 249.7 -> 236.7 mm, vias 10 -> 9
- net MISO: track 55.0 -> 66.3 mm, vias 4 -> 5
- net +3V3: track 684.8 -> 692.6 mm, vias 43 -> 45
- net IN_A1: track 92.3 -> 85.7 mm
- net N$25: track 31.4 -> 35.2 mm
- net IN_A2: track 83.7 -> 80.5 mm
- net VCC_SERVO: track 617.1 -> 619.9 mm, vias 15 -> 13
- net A1: track 85.4 -> 82.7 mm
- net BAT+: track 287.7 -> 285.5 mm
- net IN_B2: track 42.5 -> 40.5 mm
- net N$48: track 18.9 -> 17.2 mm
- net N$49: track 24.2 -> 25.6 mm
- net N$54: track 17.6 -> 18.9 mm
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Other:
- board text added: "#"
- board text added: "#____"
- board text added: "BAT 1"
- board text added: "BAT 2"
- board text added: "Created by RobotCing Team: Stanley Jochman Veronika Nemjova Designed in Slovakia Supported by Leaf"
- board text added: "IR"
- board text added: "LS"
- board text added: "Lidar"
- board text removed: "Created by RobotCing Team: Stanley Jochman Designed in Slovakia http://robotcing.sk Supported by Leaf"

Commit message: modifications
Parts:
- R17, R19: value 1k -> 10k
- moved C15 1.36 mm to (-11.3, 23.4)
- moved C24 0.90 mm to (-31.2, 28.0)
- moved U$15 0.50 mm to (24.2, 40.8)
- moved C23 0.40 mm to (-26.6, 27.5)
- moved U3 0.14 mm to (0.00, 5.80)
Routing:
- net SCL: track 221.9 -> 225.1 mm
- net N$21: track 62.0 -> 63.6 mm
- net GND: track 920.2 -> 919.0 mm
- net BAT+: track 285.5 -> 286.6 mm
- net SDA: track 236.7 -> 237.6 mm
- net +3V3: track 692.6 -> 693.5 mm
- net N$44: track 32.5 -> 31.7 mm
- net VCC_MOT: track 54.2 -> 54.9 mm

Commit message: small updates on Cing 4.1
Routing:
- net VUSB: track 34.1 -> 35.0 mm
- net MOT_B-: track 65.2 -> 65.9 mm
- net +3V3: track 693.5 -> 694.1 mm
- net N$8: track 20.0 -> 20.6 mm
