File: Hardware/Schematics/Sensors/TemperatureSensor/TemperatureSensor.brd (EAGLE design)
At the start: 15.2 x 19.1 mm, 6 parts, among them Q1 BSS138

Commit message: commit
Parts:
- removed LED1: 3mm 2ma, led:LED3MM
- removed PH1: A10, photo-elements:T0-46-A10XX
- added IC1: DS18B20, 1wire:TO92-
- added LED2: (no value), led:1206
- JP1: device pinhead:1X05 -> pinhead:1_05X2MM
- R1: value 330 -> 1k
- R2: value 1k -> 330
- moved R2 6.89 mm to (0.00, 5.83), flipped to the top, turned to 180 degrees
- moved R1 5.66 mm to (3.83, 3.87), flipped to the top, turned to 270 degrees
- moved Q1 4.62 mm to (0.00, 3.00), flipped to the top
- moved JP1 3.81 mm to (0.00, 0.00)
Connections:
- removed net N$1: JP1.5, LED1.A, PH1.2, Q1.1
- removed net N$13: JP1.1, PH1.1, R1.1
- removed net N$14: Q1.2, R1.2, R2.1
- new net 3V3: IC1.3, JP1.5, LED2.A, Q1.1, R1.1
- new net N$4: IC1.1, Q1.2, R2.1
- new net N$5: IC1.2, JP1.1, R1.2
- net N$2: now also LED2.C; no longer LED1.K
Routing:
- net N$1: track 29.8 -> 0.00 mm
- net N$13: track 12.9 -> 0.00 mm
- net N$5: track 0.00 -> 10.8 mm
- net 3V3: track 0.00 -> 8.73 mm, vias 0 -> 1
- net N$4: track 0.00 -> 8.13 mm
- net N$14: track 5.59 -> 0.00 mm
- net N$2: track 4.01 -> 2.84 mm
- net N$3: track 2.81 -> 2.00 mm
- added copper zone on layer 1, net 3V3
- added copper zone on layer 16, net GND
Other:
- board size 15.2 x 19.1 mm -> 10.2 x 12.7 mm
- board text added: "JLCPCB"
- board text added: "Sponsored"
- board text added: "by"

Commit message: gerber update
Parts:
- added U$1: TEMP-HUM-SENSOR-DHT11, diy-modules:TEMP-HUM-SENSOR-DHT11
- added U$2: OPENSOURCE, Cing Library:OSHW_5MM
- moved IC1 6.10 mm to (0.00, 14.8)
Connections:
- removed net N$4: IC1.1, Q1.2, R2.1
- removed net N$5: IC1.2, JP1.1, R1.2
- new net DATA: IC1.2, JP1.1, R1.2, U$1.2
- new net GND: IC1.1, Q1.2, R2.1, U$1.4
- net 3V3: now also U$1.1
Routing:
- net DATA: track 0.00 -> 16.4 mm
- net GND: track 0.00 -> 16.1 mm
- net N$5: track 10.8 -> 0.00 mm
- net N$4: track 8.13 -> 0.00 mm
- net 3V3: track 8.73 -> 16.6 mm, vias 1 -> 2
Other:
- board size 10.2 x 12.7 mm -> 12.2 x 18.7 mm
- board text added: "TempSensor for RobotCing"
- board text removed: "JLCPCB"
- board text removed: "Sponsored"
- board text removed: "by"
Changed lines of the file:
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@@
 <?xml version="1.0" encoding="utf-8"?>
 <!DOCTYPE eagle SYSTEM "eagle.dtd">
-<eagle version="9.2.2">
+<eagle version="9.4.0">
 <drawing>
 <settings>
@@
 <setting verticaltext="up"/>
 </settings>
-<grid distance="0.1" unitdist="mm" unit="mm" style="lines" multiple="1" display="no" altdistance="0.1" altunitdist="mm" altunit="mm"/>
+<grid distance="1" unitdist="mm" unit="mm" style="lines" multiple="1" display="no" altdistance="0.1" altunitdist="mm" altunit="mm"/>
 <layers>
 <layer number="1" name="Top" color="4" fill="1" visible="yes" active="yes"/>
@@
 <board>
 <plain>
-<wire x1="-5.1" y1="-1.1" x2="-5.1" y2="6.5" width="0.1524" layer="20"/>
-<wire x1="5.1" y1="6.5" x2="5.1" y2="-1.1" width="0.1524" layer="20"/>
-<wire x1="5.1" y1="-1.1" x2="-5.1" y2="-1.1" width="0.1524" layer="20"/>
-<wire x1="-5.1" y1="6.5" x2="5.1" y2="6.5" width="0.1524" layer="20" curve="-180"/>
-<text x="0" y="6.8" size="1.016" layer="22" rot="MR0" align="bottom-center">Sponsored</text>
-<text x="0" y="5.5" size="1.016" layer="22" rot="MR0" align="bottom-center">by</text>
-<text x="0" y="4" size="1.016" layer="22" rot="MR0" align="bottom-center">JLCPCB</text>
+<wire x1="-6.1" y1="-1.1" x2="-6.1" y2="11.5" width="0.1524" layer="20"/>
+<wire x1="6.1" y1="11.5" x2="6.1" y2="-1.1" width="0.1524" layer="20"/>
+<wire x1="6.1" y1="-1.1" x2="-6.1" y2="-1.1" width="0.1524" layer="20"/>
+<wire x1="-6.1" y1="11.5" x2="6.1" y2="11.5" width="0.1524" layer="20" curve="-180"/>
+<text x="-3.3" y="8.5" size="0.6096" layer="22" rot="MR180">TempSensor
+for RobotCing</text>
 </plain>
 <attributes>
@@
 <elements>
 <element name="R2" library="rcl" package="R1206" value="330" x="0" y="5.835" smashed="yes" rot="R180"/>
-<element name="IC1" library="1wire" package="TO92-" value="DS18B20" x="0" y="8.675" smashed="yes"/>
+<element name="IC1" library="1wire" package="TO92-" value="DS18B20" x="0" y="14.775" smashed="yes"/>
 <element name="R1" library="rcl" package="R1206" value="1k" x="3.835" y="3.865" smashed="yes" rot="R270"/>
 <element name="JP1" library="pinhead" library_urn="urn:adsk.eagle:library:325" package="1_05X2MM" package3d_urn="urn:adsk.eagle:package:22466/2" value="" x="0" y="0" smashed="yes" rot="R180">
@@
 <attribute name="VALUE" x="-1.26" y="2.23" size="1.27" layer="27" rot="R90"/>
 </element>
+<element name="U$1" library="diy-modules" package="TEMP-HUM-SENSOR-DHT11" value="TEMP-HUM-SENSOR-DHT11" x="0" y="9.6" smashed="yes" rot="R180"/>
+<element name="U$2" library="Cing Library" package="OSHW_5MM" package3d_urn="urn:adsk.eagle:package:10154747/1" value="OPENSOURCE" x="-0.1" y="4.1" smashed="yes" rot="MR0"/>
 </elements>
 <signals>
@@
 <vertex x="-6.8" y="-1.9"/>
 </polygon>
-<wire x1="2.54" y1="8.675" x2="2.1" y2="8.235" width="0.254" layer="16"/>
-<wire x1="2.1" y1="8.235" x2="2.1" y2="2.3" width="0.254" layer="16"/>
-<via x="2.1" y="2.3" extent="1-16" drill="0.6096"/>
-<wire x1="2.1" y1="2.3" x2="2.1" y2="2.85" width="0.254" layer="1"/>
-<wire x1="2.1" y1="2.85" x2="0.95" y2="4" width="0.254" layer="1"/>
+<wire x1="2.54" y1="14.775" x2="2.7" y2="14.615" width="0.254" layer="16"/>
+<wire x1="2.7" y1="14.615" x2="2.7" y2="7" width="0.254" layer="16"/>
+<wire x1="2.7" y1="7" x2="2.7" y2="2.5" width="0.254" layer="16"/>
+<wire x1="2.7" y1="2.5" x2="1.9" y2="1.7" width="0.254" layer="16"/>
+<via x="1.9" y="1.7" extent="1-16" drill="0.6096"/>
+<contactref element="U$1" pad="1"/>
+<wire x1="2.7" y1="7" x2="4" y2="7" width="0.254" layer="16"/>
+<via x="4" y="7" extent="1-16" drill="0.6096"/>
+<wire x1="4" y1="7" x2="4" y2="5.452" width="0.254" layer="1"/>
+<wire x1="4" y1="5.452" x2="3.835" y2="5.287" width="0.254" layer="1"/>
 </signal>
 <signal name="N$2">
@@
 <wire x1="-3.8" y1="5.07" x2="-3.8" y2="4.922" width="0.254" layer="1"/>
 </signal>
-<signal name="N$4">
-<contactref element="IC1" pad="1"/>
-<contactref element="R2" pad="1"/>
-<contactref element="Q1" pad="2"/>
-<wire x1="-0.2918" y1="6.873275" x2="-0.485225" y2="7.0667" width="0.254" layer="1"/>
-<wire x1="-0.485225" y1="7.0667" x2="-0.9317" y2="7.0667" width="0.254" layer="1"/>
-<wire x1="-0.9317" y1="7.0667" x2="-2.54" y2="8.675" width="0.254" layer="1"/>
-<wire x1="-0.95" y1="4" x2="-0.95" y2="4.585" width="0.254" layer="1"/>
-<wire x1="-0.95" y1="4.585" x2="-0.9317" y2="4.6033" width="0.254" layer="1"/>
-<wire x1="-0.9317" y1="4.6033" x2="-0.485225" y2="4.6033" width="0.254" layer="1"/>
-<wire x1="-0.485225" y1="4.6033" x2="-0.2918" y2="4.796725" width="0.254" layer="1"/>
-<wire x1="-0.2918" y1="4.796725" x2="-0.2918" y2="5.8" width="0.254" layer="1"/>
-<wire x1="-0.2918" y1="5.8" x2="-0.2918" y2="6.873275" width="0.254" layer="1"/>
-<wire x1="1.422" y1="5.835" x2="-0.2568" y2="5.835" width="0.254" layer="1"/>
-<wire x1="-0.2568" y1="5.835" x2="-0.2918" y2="5.8" width="0.254" layer="1"/>
-</signal>
-<signal name="N$5">
+<signal name="DATA">
 <contactref element="IC1" pad="2"/>
 <contactref element="JP1" pad="1"/>
@@
 <wire x1="3.835" y1="2.443" x2="4" y2="2.278" width="0.254" layer="1"/>
 <wire x1="4" y1="2.278" x2="4" y2="0" width="0.254" layer="1"/>
-<wire x1="2.5522" y1="6.873275" x2="2.358775" y2="7.0667" width="0.254" layer="1"/>
-<wire x1="2.358775" y1="7.0667" x2="1.6083" y2="7.0667" width="0.254" layer="1"/>
-<wire x1="1.6083" y1="7.0667" x2="0" y2="8.675" width="0.254" layer="1"/>
 <wire x1="3.835" y1="2.443" x2="3.835" y2="3.118525" width="0.254" layer="1"/>
 <wire x1="3.835" y1="3.118525" x2="2.5522" y2="4.401325" width="0.254" layer="1"/>
-<wire x1="2.5522" y1="4.401325" x2="2.5522" y2="6.873275" width="0.254" layer="1"/>
+<contactref element="U$1" pad="2"/>
+<wire x1="2.5522" y1="8.3178" x2="1.27" y2="9.6" width="0.254" layer="1"/>
+<wire x1="2.5522" y1="4.401325" x2="2.5522" y2="8.3178" width="0.254" layer="1"/>
+<wire x1="1.27" y1="9.6" x2="0" y2="10.87" width="0.254" layer="1"/>
+<wire x1="0" y1="10.87" x2="0" y2="14.775" width="0.254" layer="1"/>
 </signal>
 <signal name="N$3">
@@
 <vertex x="-7.5" y="-1.6"/>
 </polygon>
+<contactref element="IC1" pad="1"/>
+<contactref element="R2" pad="1"/>
+<contactref element="Q1" pad="2"/>
+<wire x1="-0.95" y1="4" x2="-0.95" y2="4.585" width="0.254" layer="1"/>
+<wire x1="-0.95" y1="4.585" x2="-0.9317" y2="4.6033" width="0.254" layer="1"/>
+<wire x1="-0.9317" y1="4.6033" x2="-0.485225" y2="4.6033" width="0.254" layer="1"/>
+<wire x1="-0.485225" y1="4.6033" x2="-0.2918" y2="4.796725" width="0.254" layer="1"/>
+<wire x1="-0.2918" y1="4.796725" x2="-0.2918" y2="5.8" width="0.254" layer="1"/>
+<wire x1="-0.2918" y1="5.8" x2="-0.2918" y2="6.873275" width="0.254" layer="1"/>
+<wire x1="1.422" y1="5.835" x2="-0.2568" y2="5.835" width="0.254" layer="1"/>
+<wire x1="-0.2568" y1="5.835" x2="-0.2918" y2="5.8" width="0.254" layer="1"/>
+<contactref element="U$1" pad="4"/>
+<wire x1="-0.485225" y1="7.0667" x2="-2" y2="7.0667" width="0.254" layer="1"/>
+<wire x1="-0.2918" y1="6.873275" x2="-0.485225" y2="7.0667" width="0.254" layer="1"/>
+<wire x1="-2.54" y1="7.6067" x2="-2" y2="7.0667" width="0.254" layer="1"/>
+<wire x1="-2.54" y1="7.6067" x2="-2.54" y2="9.6" width="0.254" layer="1"/>
+<wire x1="-2.54" y1="9.6" x2="-2.54" y2="14.775" width="0.254" layer="1"/>
+<wire x1="-3.81" y1="9.6" x2="-2.54" y2="9.6" width="0.254" layer="1"/>
 </signal>
 </signals>
@@
 </drawing>
 <compatibility>
+<note version="6.3" minversion="6.2.2" severity="warning">
+Since Version 6.2.2 text objects can contain more than one line,
+which will not be processed correctly with this version.
+</note>
 <note version="8.2" severity="warning">
 Since Version 8.2, EAGLE supports online libraries. The ids

Commit message: commit
Parts:
- JP1: device pinhead:1_05X2MM -> pinhead:1X05
- R1: value 1k -> 4k7
- moved LED2 0.50 mm to (-3.80, 4.00)
- moved JP1 0.20 mm to (0.00, -0.20), turned to 0 degrees
- turned R1 to 90 degrees
Routing:
- net DATA: track 16.4 -> 31.3 mm
- net 3V3: track 16.6 -> 5.70 mm, vias 2 -> 0
Other:
- board size 12.2 x 18.7 mm -> 13.2 x 20.2 mm
Changed lines of the file:
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@@
 <drawing>
 <settings>
-<setting alwaysvectorfont="no"/>
+<setting alwaysvectorfont="yes"/>
 <setting keepoldvectorfont="yes"/>
 <setting verticaltext="up"/>
 </settings>
-<grid distance="1" unitdist="mm" unit="mm" style="lines" multiple="1" display="no" altdistance="0.1" altunitdist="mm" altunit="mm"/>
+<grid distance="0.5" unitdist="mm" unit="mm" style="lines" multiple="1" display="no" altdistance="0.1" altunitdist="mm" altunit="mm"/>
 <layers>
 <layer number="1" name="Top" color="4" fill="1" visible="yes" active="yes"/>
@@
 <board>
 <plain>
-<wire x1="-6.1" y1="-1.1" x2="-6.1" y2="11.5" width="0.1524" layer="20"/>
-<wire x1="6.1" y1="11.5" x2="6.1" y2="-1.1" width="0.1524" layer="20"/>
-<wire x1="6.1" y1="-1.1" x2="-6.1" y2="-1.1" width="0.1524" layer="20"/>
-<wire x1="-6.1" y1="11.5" x2="6.1" y2="11.5" width="0.1524" layer="20" curve="-180"/>
+<wire x1="-6.6" y1="-2.1" x2="-6.6" y2="11.5" width="0.1524" layer="20"/>
+<wire x1="6.6" y1="11.5" x2="6.6" y2="-2.1" width="0.1524" layer="20"/>
+<wire x1="6.6" y1="-2.1" x2="-6.6" y2="-2.1" width="0.1524" layer="20"/>
+<wire x1="-6.6" y1="11.5" x2="6.6" y2="11.5" width="0.1524" layer="20" curve="-180"/>
 <text x="-3.3" y="8.5" size="0.6096" layer="22" rot="MR180">TempSensor
 for RobotCing</text>
@@
 <element name="R2" library="rcl" package="R1206" value="330" x="0" y="5.835" smashed="yes" rot="R180"/>
 <element name="IC1" library="1wire" package="TO92-" value="DS18B20" x="0" y="14.775" smashed="yes"/>
-<element name="R1" library="rcl" package="R1206" value="1k" x="3.835" y="3.865" smashed="yes" rot="R270"/>
-<element name="JP1" library="pinhead" library_urn="urn:adsk.eagle:library:325" package="1_05X2MM" package3d_urn="urn:adsk.eagle:package:22466/2" value="" x="0" y="0" smashed="yes" rot="R180">
-<attribute name="VALUE" x="6.35" y="3.175" size="1.27" layer="27" rot="R180"/>
+<element name="R1" library="rcl" package="R1206" value="4k7" x="3.835" y="3.865" smashed="yes" rot="R90"/>
+<element name="JP1" library="pinhead" library_urn="urn:adsk.eagle:library:325" package="1X05" package3d_urn="urn:adsk.eagle:package:22469/2" value="" x="0" y="-0.2" smashed="yes">
+<attribute name="VALUE" x="-6.35" y="-3.375" size="1.27" layer="27"/>
 </element>
 <element name="Q1" library="Cing Library" package="SOT23" value="BSS138" x="0" y="3" smashed="yes" rot="R180">
@@
 <attribute name="OC_NEWARK" value="67R2009" x="0" y="3" size="1.778" layer="27" rot="R180" display="off"/>
 </element>
-<element name="LED2" library="led" library_urn="urn:adsk.eagle:library:259" package="1206" package3d_urn="urn:adsk.eagle:package:15796/1" value="" x="-3.8" y="3.5" smashed="yes" rot="R90">
-<attribute name="VALUE" x="-1.26" y="2.23" size="1.27" layer="27" rot="R90"/>
+<element name="LED2" library="led" library_urn="urn:adsk.eagle:library:259" package="1206" package3d_urn="urn:adsk.eagle:package:15796/1" value="" x="-3.8" y="4" smashed="yes" rot="R90">
+<attribute name="VALUE" x="-1.26" y="2.73" size="1.27" layer="27" rot="R90"/>
 </element>
 <element name="U$1" library="diy-modules" package="TEMP-HUM-SENSOR-DHT11" value="TEMP-HUM-SENSOR-DHT11" x="0" y="9.6" smashed="yes" rot="R180"/>
@@
 <vertex x="-6.8" y="-1.9"/>
 </polygon>
-<wire x1="2.54" y1="14.775" x2="2.7" y2="14.615" width="0.254" layer="16"/>
-<wire x1="2.7" y1="14.615" x2="2.7" y2="7" width="0.254" layer="16"/>
-<wire x1="2.7" y1="7" x2="2.7" y2="2.5" width="0.254" layer="16"/>
-<wire x1="2.7" y1="2.5" x2="1.9" y2="1.7" width="0.254" layer="16"/>
-<via x="1.9" y="1.7" extent="1-16" drill="0.6096"/>
 <contactref element="U$1" pad="1"/>
-<wire x1="2.7" y1="7" x2="4" y2="7" width="0.254" layer="16"/>
-<via x="4" y="7" extent="1-16" drill="0.6096"/>
-<wire x1="4" y1="7" x2="4" y2="5.452" width="0.254" layer="1"/>
-<wire x1="4" y1="5.452" x2="3.835" y2="5.287" width="0.254" layer="1"/>
+<wire x1="2.54" y1="14.775" x2="3.81" y2="13.505" width="0.254" layer="1"/>
+<wire x1="3.81" y1="13.505" x2="3.81" y2="9.6" width="0.254" layer="1"/>
 </signal>
 <signal name="N$2">
@@
 <contactref element="LED2" pad="C"/>
 <wire x1="-1.422" y1="5.835" x2="-3.035" y2="5.835" width="0.254" layer="1"/>
-<wire x1="-3.035" y1="5.835" x2="-3.8" y2="5.07" width="0.254" layer="1"/>
-<wire x1="-3.8" y1="5.07" x2="-3.8" y2="4.922" width="0.254" layer="1"/>
+<wire x1="-3.035" y1="5.835" x2="-3.448" y2="5.422" width="0.254" layer="1"/>
+<wire x1="-3.448" y1="5.422" x2="-3.8" y2="5.422" width="0.254" layer="1"/>
 </signal>
 <signal name="DATA">
@@
 <contactref element="JP1" pad="1"/>
 <contactref element="R1" pad="2"/>
-<wire x1="3.835" y1="2.443" x2="4" y2="2.278" width="0.254" layer="1"/>
-<wire x1="4" y1="2.278" x2="4" y2="0" width="0.254" layer="1"/>
-<wire x1="3.835" y1="2.443" x2="3.835" y2="3.118525" width="0.254" layer="1"/>
-<wire x1="3.835" y1="3.118525" x2="2.5522" y2="4.401325" width="0.254" layer="1"/>
 <contactref element="U$1" pad="2"/>
 <wire x1="2.5522" y1="8.3178" x2="1.27" y2="9.6" width="0.254" layer="1"/>
-<wire x1="2.5522" y1="4.401325" x2="2.5522" y2="8.3178" width="0.254" layer="1"/>
 <wire x1="1.27" y1="9.6" x2="0" y2="10.87" width="0.254" layer="1"/>
 <wire x1="0" y1="10.87" x2="0" y2="14.775" width="0.254" layer="1"/>
+<wire x1="-2.129675" y1="15.7656" x2="-2.950325" y2="15.7656" width="0.254" layer="1"/>
+<wire x1="-2.950325" y1="15.7656" x2="-5.08" y2="13.635925" width="0.254" layer="1"/>
+<wire x1="0" y1="14.775" x2="-1.139075" y2="14.775" width="0.254" layer="1"/>
+<wire x1="-1.139075" y1="14.775" x2="-2.129675" y2="15.7656" width="0.254" layer="1"/>
+<wire x1="-5.08" y1="13.635925" x2="-5.08" y2="-0.2" width="0.254" layer="1"/>
+<wire x1="3.835" y1="5.287" x2="2.5522" y2="6.5698" width="0.254" layer="1"/>
+<wire x1="2.5522" y1="6.5698" x2="2.5522" y2="8.3178" width="0.254" layer="1"/>
 </signal>
 <signal name="N$3">
 <contactref element="Q1" pad="3"/>
 <contactref element="JP1" pad="3"/>
-<wire x1="0" y1="2" x2="0" y2="0" width="0.254" layer="1"/>
+<wire x1="0" y1="2" x2="0" y2="-0.2" width="0.254" layer="1"/>
 </signal>
 <signal name="GND">
 <polygon width="0.254" layer="16">
-<vertex x="-7.5" y="13.1"/>
-<vertex x="8" y="13.1"/>
-<vertex x="8" y="-1.6"/>
-<vertex x="-7.5" y="-1.6"/>
+<vertex x="-7.5" y="18.6"/>
+<vertex x="8" y="18.6"/>
+<vertex x="8" y="-2.1"/>
+<vertex x="-7.5" y="-2.1"/>
 </polygon>
 <contactref element="IC1" pad="1"/>
@@
 <mfgpreviewcolor name="substratecolor" color="0xFF786E46"/>
 </mfgpreviewcolors>
-<errors>
-</errors>
 </board>
 </drawing>
