File: Hardware/Schematics/Sensors/TemperatureSensor/TemperatureSensor.sch (EAGLE design)
At the start: 6 parts, among them IC1 DS18B20, Q1 BSS138

Commit message: commit
Parts:
- removed LED1: 3mm 2ma, led:TLLY4400
- added LED2: (no value), led:LEDSMT1206
- JP1: device pinhead:PINHD-1X5 -> pinhead:PINHD-1X55X2MM
Connections:
- removed net N$1: IC1P.VDD, JP1.5, LED1.A, Q1.G, R1.1
- new net 3V3: IC1P.VDD, JP1.5, LED2.A, Q1.G, R1.1
- net N$2: now also LED2.C; no longer LED1.C
Changed lines of the file:
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@@
 <?xml version="1.0" encoding="utf-8"?>
 <!DOCTYPE eagle SYSTEM "eagle.dtd">
-<eagle version="9.1.0">
+<eagle version="9.2.2">
 <drawing>
 <settings>
-<setting alwaysvectorfont="yes"/>
+<setting alwaysvectorfont="no"/>
 <setting keepoldvectorfont="yes"/>
 <setting verticaltext="up"/>
@@
 </classes>
 <parts>
-<part name="LED1" library="led" deviceset="TLLY4400" device="" value="3mm 2ma"/>
 <part name="R2" library="rcl" deviceset="R-EU_" device="R1206" value="330"/>
 <part name="IC1" library="1wire" deviceset="DS18B20" device=""/>
 <part name="R1" library="rcl" deviceset="R-EU_" device="R1206" value="1k"/>
-<part name="JP1" library="pinhead" library_urn="urn:adsk.eagle:library:325" deviceset="PINHD-1X5" device="" package3d_urn="urn:adsk.eagle:package:22469/2"/>
+<part name="JP1" library="pinhead" library_urn="urn:adsk.eagle:library:325" deviceset="PINHD-1X5" device="5X2MM" package3d_urn="urn:adsk.eagle:package:22466/2"/>
 <part name="Q1" library="Cing Library" deviceset="BSS138" device=""/>
+<part name="LED2" library="led" library_urn="urn:adsk.eagle:library:259" deviceset="LED" device="SMT1206" package3d_urn="urn:adsk.eagle:package:15796/1"/>
 </parts>
 <sheets>
@@
 </plain>
 <instances>
-<instance part="LED1" gate="G$1" x="12.7" y="60.96" rot="R90"/>
-<instance part="R2" gate="G$1" x="22.86" y="30.48"/>
-<instance part="IC1" gate="A" x="15.24" y="45.72" rot="R270"/>
-<instance part="IC1" gate="_1W" x="17.78" y="50.8" rot="R180"/>
-<instance part="IC1" gate="P" x="15.24" y="43.18" rot="R90"/>
-<instance part="R1" gate="G$1" x="20.32" y="55.88"/>
-<instance part="JP1" gate="A" x="17.78" y="5.08" rot="R270"/>
-<instance part="Q1" gate="G$1" x="15.24" y="17.78" rot="MR180"/>
+<instance part="R2" gate="G$1" x="22.86" y="30.48" smashed="yes">
+<attribute name="NAME" x="19.05" y="31.9786" size="1.778" layer="95"/>
+<attribute name="VALUE" x="19.05" y="27.178" size="1.778" layer="96"/>
+</instance>
+<instance part="IC1" gate="A" x="15.24" y="45.72" smashed="yes" rot="R270">
+<attribute name="NAME" x="15.875" y="40.005" size="1.778" layer="95" rot="R270"/>
+<attribute name="VALUE" x="13.335" y="40.005" size="1.778" layer="96" rot="R270"/>
+</instance>
+<instance part="IC1" gate="_1W" x="17.78" y="50.8" smashed="yes" rot="R180">
+<attribute name="NAME" x="26.67" y="48.895" size="1.778" layer="95" font="vector" rot="R180"/>
+</instance>
+<instance part="IC1" gate="P" x="15.24" y="43.18" smashed="yes" rot="R90">
+<attribute name="NAME" x="15.875" y="42.545" size="1.778" layer="95" font="vector" rot="R90"/>
+</instance>
+<instance part="R1" gate="G$1" x="20.32" y="55.88" smashed="yes">
+<attribute name="NAME" x="16.51" y="57.3786" size="1.778" layer="95"/>
+<attribute name="VALUE" x="16.51" y="52.578" size="1.778" layer="96"/>
+</instance>
+<instance part="JP1" gate="A" x="17.78" y="5.08" smashed="yes" rot="R270">
+<attribute name="NAME" x="26.035" y="11.43" size="1.778" layer="95" rot="R270"/>
+<attribute name="VALUE" x="7.62" y="11.43" size="1.778" layer="96" rot="R270"/>
+</instance>
+<instance part="Q1" gate="G$1" x="15.24" y="17.78" smashed="yes" rot="MR180">
+<attribute name="VALUE" x="3.81" y="17.78" size="1.778" layer="96" rot="MR180"/>
+<attribute name="NAME" x="3.81" y="15.24" size="1.778" layer="95" rot="MR180"/>
+</instance>
+<instance part="LED2" gate="G$1" x="12.7" y="60.96" smashed="yes" rot="R90">
+<attribute name="NAME" x="17.272" y="64.516" size="1.778" layer="95" rot="R180"/>
+<attribute name="VALUE" x="17.272" y="66.675" size="1.778" layer="96" rot="R180"/>
+</instance>
 </instances>
 <busses>
 </busses>
 <nets>
-<net name="N$1" class="0">
+<net name="3V3" class="0">
 <segment>
 <wire x1="7.62" y1="12.7" x2="12.7" y2="12.7" width="0.1524" layer="91"/>
@@
 <wire x1="7.62" y1="20.32" x2="7.62" y2="12.7" width="0.1524" layer="91"/>
 <pinref part="JP1" gate="A" pin="5"/>
-<wire x1="7.62" y1="30.48" x2="7.62" y2="20.32" width="0.1524" layer="91"/>
-<pinref part="LED1" gate="G$1" pin="A"/>
 <wire x1="10.16" y1="60.96" x2="7.62" y2="60.96" width="0.1524" layer="91"/>
-<wire x1="7.62" y1="30.48" x2="7.62" y2="43.18" width="0.1524" layer="91"/>
+<wire x1="7.62" y1="20.32" x2="7.62" y2="43.18" width="0.1524" layer="91"/>
 <pinref part="IC1" gate="P" pin="VDD"/>
 <wire x1="7.62" y1="43.18" x2="7.62" y2="55.88" width="0.1524" layer="91"/>
@@
 <wire x1="12.7" y1="20.32" x2="7.62" y2="20.32" width="0.1524" layer="91"/>
 <junction x="7.62" y="20.32"/>
+<pinref part="LED2" gate="G$1" pin="A"/>
+<label x="7.62" y="25.4" size="1.778" layer="95" rot="R180" xref="yes"/>
 </segment>
 </net>
 <net name="N$2" class="0">
 <segment>
-<pinref part="LED1" gate="G$1" pin="C"/>
 <wire x1="33.02" y1="60.96" x2="17.78" y2="60.96" width="0.1524" layer="91"/>
 <pinref part="R2" gate="G$1" pin="2"/>
 <wire x1="27.94" y1="30.48" x2="33.02" y2="30.48" width="0.1524" layer="91"/>
 <wire x1="33.02" y1="30.48" x2="33.02" y2="60.96" width="0.1524" layer="91"/>
+<pinref part="LED2" gate="G$1" pin="C"/>
 </segment>
 </net>

Commit message: gerber update
Parts:
- added U$1: TEMP-HUM-SENSOR-DHT11, diy-modules:TEMP-HUM-SENSOR-DHT11
- added U$2: OPENSOURCE, Cing Library:OPENSOURCE
Connections:
- removed net N$4: IC1P.GND, Q1.S, R2.1
- removed net N$5: IC1_1W.1W, JP1.1, R1.2
- new net DATA: IC1_1W.1W, JP1.1, R1.2, U$1.DAT
- new net GND: IC1P.GND, Q1.S, R2.1, U$1.GND
- net 3V3: now also U$1.VDD
Changed lines of the file:
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@@
 <?xml version="1.0" encoding="utf-8"?>
 <!DOCTYPE eagle SYSTEM "eagle.dtd">
-<eagle version="9.2.2">
+<eagle version="9.4.0">
 <drawing>
 <settings>
@@
 <part name="Q1" library="Cing Library" deviceset="BSS138" device=""/>
 <part name="LED2" library="led" library_urn="urn:adsk.eagle:library:259" deviceset="LED" device="SMT1206" package3d_urn="urn:adsk.eagle:package:15796/1"/>
+<part name="U$1" library="diy-modules" deviceset="TEMP-HUM-SENSOR-DHT11" device=""/>
+<part name="U$2" library="Cing Library" deviceset="OPENSOURCE" device="" package3d_urn="urn:adsk.eagle:package:10154747/1"/>
 </parts>
 <sheets>
@@
 <attribute name="VALUE" x="17.272" y="66.675" size="1.778" layer="96" rot="R180"/>
 </instance>
+<instance part="U$1" gate="G$1" x="58.42" y="38.1" smashed="yes">
+<attribute name="NAME" x="50.8" y="53.34" size="1.778" layer="95"/>
+<attribute name="VALUE" x="50.8" y="50.8" size="1.778" layer="95"/>
+</instance>
+<instance part="U$2" gate="G$1" x="-30.48" y="45.72" smashed="yes"/>
 </instances>
 <busses>
@@
 <label x="7.62" y="25.4" size="1.778" layer="95" rot="R180" xref="yes"/>
 </segment>
+<segment>
+<pinref part="U$1" gate="G$1" pin="VDD"/>
+<wire x1="45.72" y1="43.18" x2="43.18" y2="43.18" width="0.1524" layer="91"/>
+<label x="43.18" y="43.18" size="1.778" layer="95" rot="R180" xref="yes"/>
+</segment>
 </net>
 <net name="N$2" class="0">
@@
 </segment>
 </net>
-<net name="N$4" class="0">
+<net name="GND" class="0">
 <segment>
 <pinref part="IC1" gate="P" pin="GND"/>
@@
 <wire x1="17.78" y1="22.86" x2="17.78" y2="30.48" width="0.1524" layer="91"/>
 <junction x="17.78" y="30.48"/>
+<label x="22.86" y="38.1" size="1.778" layer="95" xref="yes"/>
+</segment>
+<segment>
+<pinref part="U$1" gate="G$1" pin="GND"/>
+<wire x1="45.72" y1="35.56" x2="43.18" y2="35.56" width="0.1524" layer="91"/>
+<label x="43.18" y="35.56" size="1.778" layer="95" rot="R180" xref="yes"/>
 </segment>
 </net>
-<net name="N$5" class="0">
+<net name="DATA" class="0">
 <segment>
 <pinref part="IC1" gate="_1W" pin="1W"/>
@@
 <wire x1="27.94" y1="55.88" x2="25.4" y2="55.88" width="0.1524" layer="91"/>
 <junction x="27.94" y="50.8"/>
+<label x="27.94" y="50.8" size="1.778" layer="95" xref="yes"/>
+</segment>
+<segment>
+<pinref part="U$1" gate="G$1" pin="DAT"/>
+<wire x1="45.72" y1="40.64" x2="43.18" y2="40.64" width="0.1524" layer="91"/>
+<label x="43.18" y="40.64" size="1.778" layer="95" rot="R180" xref="yes"/>
 </segment>
 </net>

Commit message: commit
Parts:
- JP1: device pinhead:PINHD-1X55X2MM -> pinhead:PINHD-1X5
- R1: value 1k -> 4k7
Changed lines of the file:
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@@
 <drawing>
 <settings>
-<setting alwaysvectorfont="no"/>
+<setting alwaysvectorfont="yes"/>
 <setting keepoldvectorfont="yes"/>
 <setting verticaltext="up"/>
@@
 <part name="R2" library="rcl" deviceset="R-EU_" device="R1206" value="330"/>
 <part name="IC1" library="1wire" deviceset="DS18B20" device=""/>
-<part name="R1" library="rcl" deviceset="R-EU_" device="R1206" value="1k"/>
-<part name="JP1" library="pinhead" library_urn="urn:adsk.eagle:library:325" deviceset="PINHD-1X5" device="5X2MM" package3d_urn="urn:adsk.eagle:package:22466/2"/>
+<part name="R1" library="rcl" deviceset="R-EU_" device="R1206" value="4k7"/>
+<part name="JP1" library="pinhead" library_urn="urn:adsk.eagle:library:325" deviceset="PINHD-1X5" device="" package3d_urn="urn:adsk.eagle:package:22469/2"/>
 <part name="Q1" library="Cing Library" deviceset="BSS138" device=""/>
 <part name="LED2" library="led" library_urn="urn:adsk.eagle:library:259" deviceset="LED" device="SMT1206" package3d_urn="urn:adsk.eagle:package:15796/1"/>
