File: Hardware/Schematics/Sensors/ShineSensor/ShineSensor.brd (EAGLE design)
At the start: 12.7 x 19.1 mm, 6 parts, among them IC1 DS18B20, Q1 BSS138

Commit message: commit
Parts:
- removed IC1: DS18B20, 1wire:TO92-
- removed LED1: 3mm 2ma, led:LED3MM
- added LED2: (no value), led:1206
- added PH1: A10, photo-elements:T0-46-A10XX
- JP1: device pinhead:1X05 -> pinhead:1_05X2MM
- R1: value 1k -> 330
- R2: value 330 -> 1k
- moved R1 7.68 mm to (3.81, 7.50), flipped to the top, turned to 90 degrees
- moved JP1 6.48 mm to (0.00, 3.81)
- moved Q1 6.36 mm to (0.00, 6.62), flipped to the top
- moved R2 4.16 mm to (0.00, 9.50), flipped to the top, turned to 180 degrees
Connections:
- removed net N$1: IC1.3, JP1.5, LED1.A, Q1.1, R1.1
- removed net N$4: IC1.1, Q1.2, R2.1
- removed net N$5: IC1.2, JP1.1, R1.2
- new net 3V3: JP1.5, LED2.A, PH1.2, Q1.1
- new net N$13: JP1.1, PH1.1, R1.1
- new net N$14: Q1.2, R1.2, R2.1
- net N$2: now also LED2.C; no longer LED1.K
Routing:
- net N$1: track 35.5 -> 0.00 mm
- net N$5: track 14.6 -> 0.00 mm
- net N$13: track 0.00 -> 13.5 mm
- net N$4: track 11.6 -> 0.00 mm
- net 3V3: track 0.00 -> 11.1 mm
- net N$14: track 0.00 -> 5.78 mm
- net N$3: track 2.81 -> 1.81 mm
- net N$2: track 3.44 -> 2.60 mm
- added copper zone on layer 1, net 3V3
- added copper zone on layer 16, net GND
Other:
- board size 12.7 x 19.1 mm -> 10.2 x 14.9 mm
- board text added: "JLCPCB"
- board text added: "Sponsored"
- board text added: "by"

Commit message: gerber update
Parts:
- added U$1: OPENSOURCE, Cing Library:OSHW_5MM
Other:
- board text added: "ShineSensor for robot Cing"
- board text removed: "JLCPCB"
- board text removed: "Sponsored"
- board text removed: "by"
Changed lines of the file:
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@@
 <?xml version="1.0" encoding="utf-8"?>
 <!DOCTYPE eagle SYSTEM "eagle.dtd">
-<eagle version="9.2.2">
+<eagle version="9.4.0">
 <drawing>
 <settings>
@@
 <wire x1="5.1" y1="2.4" x2="-5.1" y2="2.4" width="0.1524" layer="20"/>
 <wire x1="-5.1" y1="12.2" x2="5.1" y2="12.2" width="0.1524" layer="20" curve="-180"/>
-<text x="0" y="12" size="1.016" layer="22" rot="MR0" align="bottom-center">Sponsored</text>
-<text x="0" y="10.7" size="1.016" layer="22" rot="MR0" align="bottom-center">by</text>
-<text x="0" y="9.1" size="1.016" layer="22" rot="MR0" align="bottom-center">JLCPCB</text>
+<text x="4.5" y="9.4" size="0.8128" layer="22" rot="MR0">ShineSensor
+for robot Cing</text>
 </plain>
 <attributes>
@@
 <attribute name="VALUE" x="-1.24" y="6.23" size="1.27" layer="27" rot="R90"/>
 </element>
+<element name="U$1" library="Cing Library" package="OSHW_5MM" package3d_urn="urn:adsk.eagle:package:10154747/1" value="OPENSOURCE" x="0" y="6.6" smashed="yes" rot="MR0"/>
 </elements>
 <signals>
@@
 </drawing>
 <compatibility>
+<note version="6.3" minversion="6.2.2" severity="warning">
+Since Version 6.2.2 text objects can contain more than one line,
+which will not be processed correctly with this version.
+</note>
 <note version="8.2" severity="warning">
 Since Version 8.2, EAGLE supports online libraries. The ids

Commit message: gerber update
Changed lines of the file:
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@@
 <drawing>
 <settings>
-<setting alwaysvectorfont="no"/>
+<setting alwaysvectorfont="yes"/>
 <setting keepoldvectorfont="yes"/>
 <setting verticaltext="up"/>
@@
 <vertex x="11.9" y="1.4"/>
 <vertex x="11.8" y="1.3"/>
-<vertex x="-8.4" y="1.3"/>
-<vertex x="-8.6" y="1.5"/>
-<vertex x="-9.8" y="2.7"/>
+<vertex x="-9.8" y="1.3"/>
 </polygon>
 <wire x1="-1.7" y1="14" x2="-1.7" y2="6.11" width="0.254" layer="16"/>

Commit message: commit
Parts:
- JP1: device pinhead:1_05X2MM -> pinhead:1X05
- moved U$1 1.75 mm to (0.00, 8.35)
- moved LED2 0.50 mm to (-3.78, 8.00)
- moved PH1 0.50 mm to (0.00, 14.5)
- moved Q1 0.50 mm to (0.00, 7.12)
- moved R1 0.50 mm to (3.81, 8.00)
- moved R2 0.50 mm to (0.00, 10.0)
Routing:
- net N$13: track 13.5 -> 15.2 mm
- net 3V3: track 11.1 -> 12.1 mm
- net N$3: track 1.81 -> 2.31 mm
Other:
- board size 10.2 x 14.9 mm -> 12.7 x 16.7 mm
Changed lines of the file:
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@@
 <drawing>
 <settings>
-<setting alwaysvectorfont="yes"/>
+<setting alwaysvectorfont="no"/>
 <setting keepoldvectorfont="yes"/>
 <setting verticaltext="up"/>
 </settings>
-<grid distance="0.1" unitdist="mm" unit="mm" style="lines" multiple="1" display="no" altdistance="0.01" altunitdist="mm" altunit="mm"/>
+<grid distance="0.25" unitdist="mm" unit="mm" style="lines" multiple="1" display="no" altdistance="0.01" altunitdist="mm" altunit="mm"/>
 <layers>
 <layer number="1" name="Top" color="4" fill="1" visible="yes" active="yes"/>
@@
 <board>
 <plain>
-<wire x1="-5.1" y1="2.4" x2="-5.1" y2="12.2" width="0.1524" layer="20"/>
-<wire x1="5.1" y1="12.2" x2="5.1" y2="2.4" width="0.1524" layer="20"/>
-<wire x1="5.1" y1="2.4" x2="-5.1" y2="2.4" width="0.1524" layer="20"/>
-<wire x1="-5.1" y1="12.2" x2="5.1" y2="12.2" width="0.1524" layer="20" curve="-180"/>
-<text x="4.5" y="9.4" size="0.8128" layer="22" rot="MR0">ShineSensor
+<wire x1="-6.35" y1="1.9" x2="-6.35" y2="12.2" width="0.1524" layer="20"/>
+<wire x1="6.35" y1="12.2" x2="6.35" y2="1.9" width="0.1524" layer="20"/>
+<wire x1="6.35" y1="1.9" x2="-6.35" y2="1.9" width="0.1524" layer="20"/>
+<wire x1="-6.35" y1="12.2" x2="6.35" y2="12.2" width="0.1524" layer="20" curve="-180"/>
+<text x="3.5" y="11.4" size="0.8128" layer="22" rot="MR0">ShineSensor
 for robot Cing</text>
 </plain>
@@
 </autorouter>
 <elements>
-<element name="PH1" library="photo-elements" library_urn="urn:adsk.eagle:library:323" package="T0-46-A10XX" package3d_urn="urn:adsk.eagle:package:22201/1" value="A10" x="0" y="14" smashed="yes" rot="R180"/>
-<element name="R1" library="rcl" library_urn="urn:adsk.eagle:library:334" package="R1206" package3d_urn="urn:adsk.eagle:package:23540/2" value="330" x="3.815" y="7.5" smashed="yes" rot="R90">
-<attribute name="SPICEPREFIX" value="R" x="3.815" y="7.5" size="1.778" layer="27" rot="R90" display="off"/>
+<element name="PH1" library="photo-elements" library_urn="urn:adsk.eagle:library:323" package="T0-46-A10XX" package3d_urn="urn:adsk.eagle:package:22201/1" value="A10" x="0" y="14.5" smashed="yes" rot="R180"/>
+<element name="R1" library="rcl" library_urn="urn:adsk.eagle:library:334" package="R1206" package3d_urn="urn:adsk.eagle:package:23540/2" value="330" x="3.815" y="8" smashed="yes" rot="R90">
+<attribute name="SPICEPREFIX" value="R" x="3.815" y="8" size="1.778" layer="27" rot="R90" display="off"/>
 </element>
-<element name="R2" library="rcl" library_urn="urn:adsk.eagle:library:334" package="R1206" package3d_urn="urn:adsk.eagle:package:23540/2" value="1k" x="0" y="9.5" smashed="yes" rot="R180">
-<attribute name="SPICEPREFIX" value="R" x="0" y="9.5" size="1.778" layer="27" rot="R180" display="off"/>
+<element name="R2" library="rcl" library_urn="urn:adsk.eagle:library:334" package="R1206" package3d_urn="urn:adsk.eagle:package:23540/2" value="1k" x="0" y="10" smashed="yes" rot="R180">
+<attribute name="SPICEPREFIX" value="R" x="0" y="10" size="1.778" layer="27" rot="R180" display="off"/>
 </element>
-<element name="JP1" library="pinhead" library_urn="urn:adsk.eagle:library:325" package="1_05X2MM" package3d_urn="urn:adsk.eagle:package:22466/2" value="" x="0" y="3.81" smashed="yes" rot="R180">
+<element name="JP1" library="pinhead" library_urn="urn:adsk.eagle:library:325" package="1X05" package3d_urn="urn:adsk.eagle:package:22469/2" value="" x="0" y="3.81" smashed="yes" rot="R180">
+<attribute name="POPULARITY" value="69" x="0" y="3.81" size="1.778" layer="27" rot="R180" display="off"/>
 <attribute name="VALUE" x="-8.255" y="7.62" size="1.27" layer="27" rot="R270"/>
 </element>
-<element name="Q1" library="Cing Library" package="SOT23" value="BSS138" x="0" y="6.62" smashed="yes" rot="R180">
-<attribute name="MF" value="Fairchild" x="0" y="6.62" size="1.778" layer="27" rot="R180" display="off"/>
-<attribute name="MPN" value="BSS138" x="0" y="6.62" size="1.778" layer="27" rot="R180" display="off"/>
-<attribute name="OC_FARNELL" value="9845330" x="0" y="6.62" size="1.778" layer="27" rot="R180" display="off"/>
-<attribute name="OC_NEWARK" value="67R2009" x="0" y="6.62" size="1.778" layer="27" rot="R180" display="off"/>
+<element name="Q1" library="Cing Library" package="SOT23" value="BSS138" x="0" y="7.12" smashed="yes" rot="R180">
+<attribute name="MF" value="Fairchild" x="0" y="7.12" size="1.778" layer="27" rot="R180" display="off"/>
+<attribute name="MPN" value="BSS138" x="0" y="7.12" size="1.778" layer="27" rot="R180" display="off"/>
+<attribute name="OC_FARNELL" value="9845330" x="0" y="7.12" size="1.778" layer="27" rot="R180" display="off"/>
+<attribute name="OC_NEWARK" value="67R2009" x="0" y="7.12" size="1.778" layer="27" rot="R180" display="off"/>
 </element>
-<element name="LED2" library="led" library_urn="urn:adsk.eagle:library:259" package="1206" package3d_urn="urn:adsk.eagle:package:15796/1" value="" x="-3.78" y="7.5" smashed="yes" rot="R90">
-<attribute name="VALUE" x="-1.24" y="6.23" size="1.27" layer="27" rot="R90"/>
+<element name="LED2" library="led" library_urn="urn:adsk.eagle:library:259" package="1206" package3d_urn="urn:adsk.eagle:package:15796/1" value="" x="-3.78" y="8" smashed="yes" rot="R90">
+<attribute name="VALUE" x="-1.24" y="6.73" size="1.27" layer="27" rot="R90"/>
 </element>
-<element name="U$1" library="Cing Library" package="OSHW_5MM" package3d_urn="urn:adsk.eagle:package:10154747/1" value="OPENSOURCE" x="0" y="6.6" smashed="yes" rot="MR0"/>
+<element name="U$1" library="Cing Library" package="OSHW_5MM" package3d_urn="urn:adsk.eagle:package:10154747/1" value="OPENSOURCE" x="0" y="8.35" smashed="yes" rot="MR0"/>
 </elements>
 <signals>
@@
 <contactref element="R1" pad="1"/>
 <contactref element="JP1" pad="1"/>
-<wire x1="4" y1="3.81" x2="4" y2="5.893" width="0.254" layer="1"/>
-<wire x1="4" y1="5.893" x2="3.815" y2="6.078" width="0.254" layer="1"/>
-<wire x1="1.7" y1="14" x2="1.7" y2="6.11" width="0.254" layer="16"/>
-<wire x1="1.7" y1="6.11" x2="4" y2="3.81" width="0.254" layer="16"/>
+<wire x1="5.08" y1="3.81" x2="3.90015625" y2="6.08556875" width="0.254" layer="1"/>
+<wire x1="3.90015625" y1="6.08556875" x2="3.815" y2="6.578" width="0.254" layer="1"/>
+<wire x1="5.08" y1="3.81" x2="1.7" y2="7.19" width="0.254" layer="16"/>
+<wire x1="1.7" y1="7.19" x2="1.7" y2="14.5" width="0.254" layer="16"/>
 </signal>
 <signal name="N$14">
@@
 <contactref element="R2" pad="1"/>
 <contactref element="Q1" pad="2"/>
-<wire x1="1.422" y1="9.5" x2="3.237" y2="9.5" width="0.254" layer="1"/>
-<wire x1="3.237" y1="9.5" x2="3.815" y2="8.922" width="0.254" layer="1"/>
-<wire x1="1.422" y1="9.5" x2="-0.458" y2="7.62" width="0.254" layer="1"/>
-<wire x1="-0.458" y1="7.62" x2="-0.95" y2="7.62" width="0.254" layer="1"/>
+<wire x1="1.422" y1="10" x2="3.237" y2="10" width="0.254" layer="1"/>
+<wire x1="3.237" y1="10" x2="3.815" y2="9.422" width="0.254" layer="1"/>
+<wire x1="-0.95" y1="8.12" x2="-0.458" y2="8.12" width="0.254" layer="1"/>
+<wire x1="1.422" y1="10" x2="-0.458" y2="8.12" width="0.254" layer="1"/>
 </signal>
 <signal name="3V3">
@@
 <vertex x="-9.8" y="1.3"/>
 </polygon>
-<wire x1="-1.7" y1="14" x2="-1.7" y2="6.11" width="0.254" layer="16"/>
-<wire x1="-1.7" y1="6.11" x2="-4" y2="3.81" width="0.254" layer="16"/>
+<wire x1="-5.08" y1="3.81" x2="-1.7" y2="7.19" width="0.254" layer="16"/>
+<wire x1="-1.7" y1="7.19" x2="-1.7" y2="14.5" width="0.254" layer="16"/>
 </signal>
 <signal name="N$2">
 <contactref element="R2" pad="2"/>
 <contactref element="LED2" pad="C"/>
-<wire x1="-3.78" y1="8.922" x2="-3.202" y2="9.5" width="0.254" layer="1"/>
-<wire x1="-3.202" y1="9.5" x2="-1.422" y2="9.5" width="0.254" layer="1"/>
+<wire x1="-3.78" y1="9.422" x2="-3.202" y2="10" width="0.254" layer="1"/>
+<wire x1="-3.202" y1="10" x2="-1.422" y2="10" width="0.254" layer="1"/>
 </signal>
 <signal name="N$3">
 <contactref element="Q1" pad="3"/>
 <contactref element="JP1" pad="3"/>
-<wire x1="0" y1="5.62" x2="0" y2="3.81" width="0.254" layer="1"/>
+<wire x1="0" y1="6.12" x2="0" y2="3.81" width="0.254" layer="1"/>
 </signal>
 <signal name="GND">
@@
 <mfgpreviewcolor name="substratecolor" color="0xFF786E46"/>
 </mfgpreviewcolors>
-<errors>
-</errors>
 </board>
 </drawing>
