File: Hardware/Schematics/Sensors/ShineSensor/ShineSensor.sch (EAGLE design)
At the start: 6 parts, among them Q1 BSS138

Commit message: commit
Parts:
- removed LED1: 3mm 2ma, led:TLLY4400
- added LED2: (no value), led:LEDSMT1206
- JP1: device pinhead:PINHD-1X5 -> pinhead:PINHD-1X55X2MM
Connections:
- removed net N$1: JP1.5, LED1.A, PH1.2, Q1.G
- new net 3V3: JP1.5, LED2.A, PH1.2, Q1.G
- net N$2: now also LED2.C; no longer LED1.C
Changed lines of the file:
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@@
 <?xml version="1.0" encoding="utf-8"?>
 <!DOCTYPE eagle SYSTEM "eagle.dtd">
-<eagle version="9.1.0">
+<eagle version="9.2.2">
 <drawing>
 <settings>
-<setting alwaysvectorfont="yes"/>
+<setting alwaysvectorfont="no"/>
 <setting keepoldvectorfont="yes"/>
 <setting verticaltext="up"/>
@@
 <part name="PH1" library="photo-elements" library_urn="urn:adsk.eagle:library:323" deviceset="A10" device="" package3d_urn="urn:adsk.eagle:package:22201/1" technology="50_11" value="A10"/>
 <part name="R1" library="rcl" library_urn="urn:adsk.eagle:library:334" deviceset="R-EU_" device="R1206" package3d_urn="urn:adsk.eagle:package:23540/2" value="330"/>
-<part name="LED1" library="led" library_urn="urn:adsk.eagle:library:259" deviceset="TLLY4400" device="" package3d_urn="urn:adsk.eagle:package:15797/1" value="3mm 2ma"/>
 <part name="R2" library="rcl" library_urn="urn:adsk.eagle:library:334" deviceset="R-EU_" device="R1206" package3d_urn="urn:adsk.eagle:package:23540/2" value="1k"/>
-<part name="JP1" library="pinhead" library_urn="urn:adsk.eagle:library:325" deviceset="PINHD-1X5" device="" package3d_urn="urn:adsk.eagle:package:22469/2"/>
+<part name="JP1" library="pinhead" library_urn="urn:adsk.eagle:library:325" deviceset="PINHD-1X5" device="5X2MM" package3d_urn="urn:adsk.eagle:package:22466/2"/>
 <part name="Q1" library="Cing Library" deviceset="BSS138" device=""/>
+<part name="LED2" library="led" library_urn="urn:adsk.eagle:library:259" deviceset="LED" device="SMT1206" package3d_urn="urn:adsk.eagle:package:15796/1"/>
 </parts>
 <sheets>
@@
 </plain>
 <instances>
-<instance part="PH1" gate="G$1" x="12.7" y="35.56" rot="R270"/>
-<instance part="R1" gate="G$1" x="17.78" y="22.86" rot="R270"/>
-<instance part="LED1" gate="G$1" x="12.7" y="45.72" rot="R90"/>
-<instance part="R2" gate="G$1" x="22.86" y="15.24"/>
-<instance part="JP1" gate="A" x="17.78" y="-7.62" rot="R270"/>
-<instance part="Q1" gate="G$1" x="15.24" y="7.62" rot="MR180"/>
+<instance part="PH1" gate="G$1" x="12.7" y="35.56" smashed="yes" rot="R270">
+<attribute name="NAME" x="12.7" y="33.02" size="1.778" layer="95" rot="R270"/>
+<attribute name="VALUE" x="10.16" y="33.02" size="1.778" layer="96" rot="R270"/>
+</instance>
+<instance part="R1" gate="G$1" x="17.78" y="22.86" smashed="yes" rot="R270">
+<attribute name="NAME" x="19.2786" y="26.67" size="1.778" layer="95" rot="R270"/>
+<attribute name="VALUE" x="14.478" y="26.67" size="1.778" layer="96" rot="R270"/>
+</instance>
+<instance part="R2" gate="G$1" x="22.86" y="15.24" smashed="yes">
+<attribute name="NAME" x="19.05" y="16.7386" size="1.778" layer="95"/>
+<attribute name="VALUE" x="19.05" y="11.938" size="1.778" layer="96"/>
+</instance>
+<instance part="JP1" gate="A" x="17.78" y="-7.62" smashed="yes" rot="R270">
+<attribute name="NAME" x="26.035" y="-1.27" size="1.778" layer="95" rot="R270"/>
+<attribute name="VALUE" x="7.62" y="-1.27" size="1.778" layer="96" rot="R270"/>
+</instance>
+<instance part="Q1" gate="G$1" x="15.24" y="7.62" smashed="yes" rot="MR180">
+<attribute name="VALUE" x="3.81" y="7.62" size="1.778" layer="96" rot="MR180"/>
+<attribute name="NAME" x="3.81" y="5.08" size="1.778" layer="95" rot="MR180"/>
+</instance>
+<instance part="LED2" gate="G$1" x="12.7" y="45.72" smashed="yes" rot="R90">
+<attribute name="NAME" x="17.272" y="49.276" size="1.778" layer="95" rot="R180"/>
+<attribute name="VALUE" x="17.272" y="51.435" size="1.778" layer="96" rot="R180"/>
+</instance>
 </instances>
 <busses>
@@
 </segment>
 </net>
-<net name="N$1" class="0">
+<net name="3V3" class="0">
 <segment>
 <pinref part="PH1" gate="G$1" pin="2"/>
-<pinref part="LED1" gate="G$1" pin="A"/>
 <wire x1="10.16" y1="45.72" x2="7.62" y2="45.72" width="0.1524" layer="91"/>
 <wire x1="7.62" y1="45.72" x2="7.62" y2="35.56" width="0.1524" layer="91"/>
@@
 <junction x="12.7" y="10.16"/>
 <wire x1="7.62" y1="35.56" x2="7.62" y2="12.7" width="0.1524" layer="91"/>
+<pinref part="LED2" gate="G$1" pin="A"/>
+<label x="7.62" y="12.7" size="1.778" layer="95" rot="R180" xref="yes"/>
 </segment>
 </net>
@@
 <segment>
 <pinref part="R2" gate="G$1" pin="2"/>
-<pinref part="LED1" gate="G$1" pin="C"/>
 <wire x1="27.94" y1="15.24" x2="27.94" y2="45.72" width="0.1524" layer="91"/>
 <wire x1="27.94" y1="45.72" x2="17.78" y2="45.72" width="0.1524" layer="91"/>
-</segment>
-</net>
+<pinref part="LED2" gate="G$1" pin="C"/>
+</segment>
+</net>

Commit message: gerber update
Parts:
- added U$1: OPENSOURCE, Cing Library:OPENSOURCE
Changed lines of the file:
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@@
 <?xml version="1.0" encoding="utf-8"?>
 <!DOCTYPE eagle SYSTEM "eagle.dtd">
-<eagle version="9.2.2">
+<eagle version="9.4.0">
 <drawing>
 <settings>
@@
 <part name="Q1" library="Cing Library" deviceset="BSS138" device=""/>
 <part name="LED2" library="led" library_urn="urn:adsk.eagle:library:259" deviceset="LED" device="SMT1206" package3d_urn="urn:adsk.eagle:package:15796/1"/>
+<part name="U$1" library="Cing Library" deviceset="OPENSOURCE" device="" package3d_urn="urn:adsk.eagle:package:10154747/1"/>
 </parts>
 <sheets>
@@
 <attribute name="VALUE" x="17.272" y="51.435" size="1.778" layer="96" rot="R180"/>
 </instance>
+<instance part="U$1" gate="G$1" x="-20.32" y="27.94" smashed="yes"/>
 </instances>
 <busses>

Commit message: commit
Parts:
- JP1: device pinhead:PINHD-1X55X2MM -> pinhead:PINHD-1X5
Changed lines of the file:
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@@
 <part name="R1" library="rcl" library_urn="urn:adsk.eagle:library:334" deviceset="R-EU_" device="R1206" package3d_urn="urn:adsk.eagle:package:23540/2" value="330"/>
 <part name="R2" library="rcl" library_urn="urn:adsk.eagle:library:334" deviceset="R-EU_" device="R1206" package3d_urn="urn:adsk.eagle:package:23540/2" value="1k"/>
-<part name="JP1" library="pinhead" library_urn="urn:adsk.eagle:library:325" deviceset="PINHD-1X5" device="5X2MM" package3d_urn="urn:adsk.eagle:package:22466/2"/>
+<part name="JP1" library="pinhead" library_urn="urn:adsk.eagle:library:325" deviceset="PINHD-1X5" device="" package3d_urn="urn:adsk.eagle:package:22469/2"/>
 <part name="Q1" library="Cing Library" deviceset="BSS138" device=""/>
 <part name="LED2" library="led" library_urn="urn:adsk.eagle:library:259" deviceset="LED" device="SMT1206" package3d_urn="urn:adsk.eagle:package:15796/1"/>
